File: scheme/cpu.kicad_sch (KiCad schematic)
At the start: 15 parts, among them U101 STM32G0B1CCT6, Y101 32.768kHz

Commit message: feat(schematic): add MPN/LCSC fields and fix Q201 pinout
Подготовка к заказу сборки на JLCPCB:
- всем монтируемым символам добавлено скрытое поле LCSC (коды
  проверены через API JLCPCB, по возможности Basic);
- LSE Y101: Epson FC-135 CL 7 пФ (Q13FC13500002), C106/C108 6.8p C0G,
  footprint под ручную пайку; в SDK нужен LSEDRV=10;
- бусины: FB101/FB401 GZ2012D601TF, FB301 BLM21PG221SN1D (2 А);
- Y401 25 МГц X49SD25MSD2SC (CL 20 пФ), C401/C402 27p -> 33p;
- Y201 8 МГц X49SD8MSD2SC, нагрузочные 22p оставлены (предел F103
  25 пФ, сдвиг частоты для USB FS несущественен);
- C505 100n на ~CARD_DET (антидребезг), ссылка на чертёж Hirose.

Исправления:
- Q201: символ SS9013 с распиновкой TO-92 (1=E 2=B 3=C) стоял на
  footprint SOT-23 (1=B 2=E 3=C) - транзистор встал бы неправильно.
  Заменён на MMBT3904 (SOT-23, Basic), цепи B/E/C сохранены;
- лист leds переведён с 1206 на 0805, R701/R702 630 -> 680 Ом
  (630 нет в E24), LD702 ORANGE -> RED;
- C301 (DNP) получил номинал 4.7n, опечатка 25Mhz в Y401.

ERC: 0 ошибок, 0 предупреждений.
Parts:
- C101, C102, C103, C105, C107: LCSC (none) -> C49678
- C104: LCSC (none) -> C1779
- C106, C108: value 8.2p C0G -> 6.8p C0G; LCSC (none) -> C1832
- C109: LCSC (none) -> C28323
- FB101: value BLM21PG221SN1D -> 600R@100MHz 0.5A; LCSC (none) -> C1017; MPN (none) -> GZ2012D601TF
- JP101: LCSC (none) -> C42431798
- R101: LCSC (none) -> C17513
- RV101: LCSC (none) -> C36376
- U101: LCSC (none) -> C5270241
- Y101: value 32.768kHz -> 32.768kHz CL7pF; footprint Crystal:Crystal_SMD_3215-2Pin_3.2x1.5mm -> Crystal:Crystal_SMD_G8-2Pin_3.2x1.5mm_HandSoldering; LCSC (none) -> C48615; MPN FC-135 32.768kHz CL7pF -> Q13FC13500002
Other:
- note added: "LSE: Y101 32.768 кГц Epson FC-135 Q13FC13500002, 3.2x1.5 мм: CL = 7 пФ, ESR <= 70 кОм, C0 = 1.0 пФ тип. (даташит Epson FC-135, ~/Downloads/parts/xtal/). C106/C108 = 2 x (CL - Cstray) = 2 x (7 - ~3.6) ~ 6.8 пФ C0G (Cstray - выводы + дорожки, оценка). Критерий DS13560 табл. 43: gm_crit кварца <= Gmcritmax. gm_crit = 4 x ESR x (2pi f)^2 x (C0 + CL)^2 = 4 x 70k x (2pi x 32768)^2 x ((1..1.3)p + 7p)^2 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"
- note removed: "LSE: Y101 32.768 кГц 3215, CL = 7 пФ. C106/C108 = 2 x (CL - Cs) = 2 x (7 - ~3) = 8 пФ -> 8.2 пФ C0G (Cs - выводы + дорожки, оценка). Критерий DS13560 табл. 43: gm_crit кварца <= Gmcritmax. gm_crit = 4 x ESR x (2pi f)^2 x (C0 + CL)^2 = 4 x 70k x (2pi x 32768)^2 x (1p + 7p)^2 ~ 0.76 мкА/В (ESR 70 кОм - max по дистрибьютору для FC-135, C0 = 1 пФ - ПРЕДПОЛОЖЕНИЕ, проверить по DS кварца). LSEDRV = 01 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"
Changed lines of the file:
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@@
 		)
 	)
-	(text "LSE: Y101 32.768 кГц 3215, CL = 7 пФ. C106/C108 = 2 x (CL - Cs) = 2 x (7 - ~3) = 8 пФ -> 8.2 пФ C0G\n(Cs - выводы + дорожки, оценка). Критерий DS13560 табл. 43: gm_crit кварца <= Gmcritmax.\ngm_crit = 4 x ESR x (2pi f)^2 x (C0 + CL)^2 = 4 x 70k x (2pi x 32768)^2 x (1p + 7p)^2 ~ 0.76 мкА/В\n(ESR 70 кОм - max по дистрибьютору для FC-135, C0 = 1 пФ - ПРЕДПОЛОЖЕНИЕ, проверить по DS кварца).\nLSEDRV = 01 (0.75) - на грани; ставить LSEDRV = 10 (1.7 мкА/В) или 11 (2.7).\nКварц и C106/C108 вплотную к выв. 2/3, без дорожек под кварцем (DS13560 §5.3.7, AN2867)."
+	(text "LSE: Y101 32.768 кГц Epson FC-135 Q13FC13500002, 3.2x1.5 мм: CL = 7 пФ, ESR <= 70 кОм, C0 = 1.0 пФ тип.\n(даташит Epson FC-135, ~/Downloads/parts/xtal/). C106/C108 = 2 x (CL - Cstray) = 2 x (7 - ~3.6) ~ 6.8 пФ C0G\n(Cstray - выводы + дорожки, оценка). Критерий DS13560 табл. 43: gm_crit кварца <= Gmcritmax.\ngm_crit = 4 x ESR x (2pi f)^2 x (C0 + CL)^2 = 4 x 70k x (2pi x 32768)^2 x ((1..1.3)p + 7p)^2 ~ 0.76..0.82 мкА/В.\nLSEDRV = 01 (Gmcritmax 0.75 мкА/В) мало. В прошивке SDK выставить LSEDRV = 10 (medium-high, 1.7 мкА/В), запас ~2.\nАльтернатива для закупки в РФ: FC-135 32.7680KA-A3 (CL 12.5 пФ) -> C = 18 пФ и LSEDRV = 11 (2.7), запас лишь ~1.2.\nКварц и C106/C108 вплотную к выв. 2/3, без дорожек под кварцем (DS13560 §5.3.7, AN2867)."
 		(exclude_from_sim no)
 		(at 20.32 144.78 0)
@@
 			)
 		)
+		(property "LCSC" "C49678"
+			(at 137.16 59.69 0)
+			(hide yes)
+			(show_name no)
+			(do_not_autoplace no)
+			(effects
+				(font
+					(size 1.27 1.27)
+				)
+			)
+		)
 		(pin "1"
 		)
@@
 			)
 		)
+		(property "LCSC" "C1779"
+			(at 96.52 59.69 0)
+			(hide yes)
+			(show_name no)
+			(do_not_autoplace no)
+			(effects
+				(font
+					(size 1.27 1.27)
+				)
+			)
+		)
 		(pin "1"
 		)
@@
 			)
 		)
+		(property "LCSC" "C42431798"
+			(at 63.5 40.64 0)
+			(hide yes)
+			(show_name no)
+			(do_not_autoplace no)
+			(effects
+				(font
+					(size 1.27 1.27)
+				)
+			)
+		)
 		(pin "1"
 		)
@@
 			)
 		)
+		(property "LCSC" "C36376"
+			(at 45.72 128.27 0)
+			(hide yes)
+			(show_name no)
+			(do_not_autoplace no)
+			(effects
+				(font
+					(size 1.27 1.27)
+				)
+			)
+		)
 		(pin "1"
 		)
@@
 			)
 		)
+		(property "LCSC" "C49678"
+			(at 88.9 132.08 0)
+			(hide yes)
+			(show_name no)
+			(do_not_autoplace no)
+			(effects
+				(font
+					(size 1.27 1.27)
+				)
+			)
+		)
 		(pin "1"
 		)
@@
 			)
 		)
-		(property "Value" "8.2p C0G"
+		(property "Value" "6.8p C0G"
 			(at 144.78 137.16 0)
 			(show_name no)
@@
 			)
 		)
+		(property "LCSC" "C1832"
+			(at 142.24 135.89 0)
+			(hide yes)
+			(show_name no)
+			(do_not_autoplace no)
+			(effects
+				(font
+					(size 1.27 1.27)
+				)
+			)
+		)
 		(pin "1"
 		)
@@
 			)
 		)
+		(property "LCSC" "C5270241"
+			(at 203.2 139.7 0)
+			(hide yes)
+			(show_name no)
+			(do_not_autoplace no)
+			(effects
+				(font
+					(size 1.27 1.27)
+				)
+			)
+		)
 		(pin "1"
 		)
@@
 			)
 		)
+		(property "LCSC" "C49678"
+			(at 83.82 59.69 0)
+			(hide yes)
+			(show_name no)
+			(do_not_autoplace no)
+			(effects
+				(font
+					(size 1.27 1.27)
+				)
+			)
+		)
 		(pin "1"
 		)
@@
 			)
 		)
-		(property "Value" "32.768kHz"
+		(property "Value" "32.768kHz CL7pF"
 			(at 133.35 127 0)
 			(show_name no)
@@
 			)
 		)
-		(property "Footprint" "Crystal:Crystal_SMD_3215-2Pin_3.2x1.5mm"
+		(property "Footprint" "Crystal:Crystal_SMD_G8-2Pin_3.2x1.5mm_HandSoldering"
 			(at 133.35 132.08 0)
 			(hide yes)
@@
 			)
 		)
-		(property "Description" "Кварц 32.768 кГц 3.2x1.5 мм, CL = 7 пФ, ESR <= 70 кОм (напр. Epson FC-135, суффикс с CL=7 пФ уточнить)"
+		(property "Description" "Кварц 32.768 кГц 3.2x1.5 мм, Epson FC-135 (Q13FC13500002): CL 7 пФ, ESR <= 70 кОм, C0 1.0 пФ тип."
 			(at 133.35 132.08 0)
 			(hide yes)
@@
 			)
 		)
-		(property "MPN" "FC-135 32.768kHz CL7pF"
+		(property "MPN" "Q13FC13500002"
+			(at 133.35 132.08 0)
+			(hide yes)
+			(show_name no)
+			(do_not_autoplace no)
+			(effects
+				(font
+					(size 1.27 1.27)
+				)
+			)
+		)
+		(property "LCSC" "C48615"
 			(at 133.35 132.08 0)
 			(hide yes)
@@
 			)
 		)
+		(property "LCSC" "C49678"
+			(at 109.22 59.69 0)
+			(hide yes)
+			(show_name no)
+			(do_not_autoplace no)
+			(effects
+				(font
+					(size 1.27 1.27)
+				)
+			)
+		)
 		(pin "1"
 		)
@@
 			)
 		)
+		(property "LCSC" "C49678"
+			(at 66.04 132.08 0)
+			(hide yes)
+			(show_name no)
+			(do_not_autoplace no)
+			(effects
+				(font
+					(size 1.27 1.27)
+				)
+			)
+		)
 		(pin "1"
 		)
@@
 			)
 		)
-		(property "Value" "BLM21PG221SN1D"
+		(property "Value" "600R@100MHz 0.5A"
 			(at 125.73 50.8 90)
 			(show_name no)
@@
 			)
 		)
-		(property "Description" "Ферритовая бусина 220 Ом @100 МГц, 0805 (MPN - пример, проверить Rdc/ток)"
+		(property "Description" "Ферритовая бусина 600 Ом @100 МГц, 0.5 А, Rdc 0.3 Ом, 0805 (Sunlord GZ2012D601TF)"
+			(at 125.73 55.88 0)
+			(hide yes)
+			(show_name no)
+			(do_not_autoplace no)
+			(effects
+				(font
+					(size 1.27 1.27)
+				)
+			)
+		)
+		(property "MPN" "GZ2012D601TF"
+			(at 125.73 55.88 0)
+			(hide yes)
+			(show_name no)
+			(do_not_autoplace no)
+			(effects
+				(font
+					(size 1.27 1.27)
+				)
+			)
+		)
+		(property "LCSC" "C1017"
 			(at 125.73 55.88 0)
 			(hide yes)
@@
 			)
 		)
+		(property "LCSC" "C28323"
+			(at 149.86 59.69 0)
+			(hide yes)
+			(show_name no)
+			(do_not_autoplace no)
+			(effects
+				(font
+					(size 1.27 1.27)
+				)
+			)
+		)
 		(pin "1"
 		)
@@
 			)
 		)
-		(property "Value" "8.2p C0G"
+		(property "Value" "6.8p C0G"
 			(at 121.92 137.16 0)
 			(show_name no)
@@
 			)
 		)
+		(property "LCSC" "C1832"
+			(at 124.46 135.89 0)
+			(hide yes)
+			(show_name no)
+			(do_not_autoplace no)
+			(effects
+				(font
+					(size 1.27 1.27)
+				)
+			)
+		)
 		(pin "1"
 		)
@@
 			(at 57.15 128.27 0)
 			(hide yes)
+			(show_name no)
+			(do_not_autoplace no)
+			(effects
+				(font
+					(size 1.27 1.27)
+				)
+			)
+		)
+		(property "LCSC" "C17513"
+			(at 57.15 128.27 0)
+			(hide yes)
