File: scheme/w32.kicad_sch (KiCad schematic)
At the start: 23 parts, among them J501 DM3AT-SF-PEJM5, U501 W25Q32JVSSIQ

Commit message: feat(schematic): add MPN/LCSC fields and fix Q201 pinout
Подготовка к заказу сборки на JLCPCB:
- всем монтируемым символам добавлено скрытое поле LCSC (коды
  проверены через API JLCPCB, по возможности Basic);
- LSE Y101: Epson FC-135 CL 7 пФ (Q13FC13500002), C106/C108 6.8p C0G,
  footprint под ручную пайку; в SDK нужен LSEDRV=10;
- бусины: FB101/FB401 GZ2012D601TF, FB301 BLM21PG221SN1D (2 А);
- Y401 25 МГц X49SD25MSD2SC (CL 20 пФ), C401/C402 27p -> 33p;
- Y201 8 МГц X49SD8MSD2SC, нагрузочные 22p оставлены (предел F103
  25 пФ, сдвиг частоты для USB FS несущественен);
- C505 100n на ~CARD_DET (антидребезг), ссылка на чертёж Hirose.

Исправления:
- Q201: символ SS9013 с распиновкой TO-92 (1=E 2=B 3=C) стоял на
  footprint SOT-23 (1=B 2=E 3=C) - транзистор встал бы неправильно.
  Заменён на MMBT3904 (SOT-23, Basic), цепи B/E/C сохранены;
- лист leds переведён с 1206 на 0805, R701/R702 630 -> 680 Ом
  (630 нет в E24), LD702 ORANGE -> RED;
- C301 (DNP) получил номинал 4.7n, опечатка 25Mhz в Y401.

ERC: 0 ошибок, 0 предупреждений.
Parts:
- added C505: 100n, Capacitor_SMD:C_0805_2012Metric, symbol Device:C
- C501, C503: LCSC (none) -> C49678
- C502, C504: LCSC (none) -> C15850
- J501: LCSC (none) -> C114218
- R501, R502, R503, R504, R507, R508, R509, R510: LCSC (none) -> C17415
- R505, R511, R516, R517: LCSC (none) -> C17414
- R506, R512, R513, R514, R515: LCSC (none) -> C17713
- U501: LCSC (none) -> C179173
Connections:
- net GND: now also C505.2
- net ~{CARD_DET}: now also C505.1
Other:
- note added: "C505 100n (у J501, /CARD_DET -> GND): антидребезг детекта карты, RC = 47k (R506) · 100n ≈ 4.7 мс. Необязателен при программной фильтрации /CARD_DET (инженерная оценка, не из DS)."
