File: scheme/ft232rl.kicad_sch (KiCad schematic)
At the start: 20 parts, among them J301 USB_B_Mini, U301 USBLC6-2SC6, U302 FT232RL

Commit message: feat(schematic): add MPN/LCSC fields and fix Q201 pinout
Подготовка к заказу сборки на JLCPCB:
- всем монтируемым символам добавлено скрытое поле LCSC (коды
  проверены через API JLCPCB, по возможности Basic);
- LSE Y101: Epson FC-135 CL 7 пФ (Q13FC13500002), C106/C108 6.8p C0G,
  footprint под ручную пайку; в SDK нужен LSEDRV=10;
- бусины: FB101/FB401 GZ2012D601TF, FB301 BLM21PG221SN1D (2 А);
- Y401 25 МГц X49SD25MSD2SC (CL 20 пФ), C401/C402 27p -> 33p;
- Y201 8 МГц X49SD8MSD2SC, нагрузочные 22p оставлены (предел F103
  25 пФ, сдвиг частоты для USB FS несущественен);
- C505 100n на ~CARD_DET (антидребезг), ссылка на чертёж Hirose.

Исправления:
- Q201: символ SS9013 с распиновкой TO-92 (1=E 2=B 3=C) стоял на
  footprint SOT-23 (1=B 2=E 3=C) - транзистор встал бы неправильно.
  Заменён на MMBT3904 (SOT-23, Basic), цепи B/E/C сохранены;
- лист leds переведён с 1206 на 0805, R701/R702 630 -> 680 Ом
  (630 нет в E24), LD702 ORANGE -> RED;
- C301 (DNP) получил номинал 4.7n, опечатка 25Mhz в Y401.

ERC: 0 ошибок, 0 предупреждений.
Parts:
- C301: value DNP -> 4.7n; LCSC (none) -> C1744
- C302: LCSC (none) -> C1710
- C303, C304, C305: LCSC (none) -> C49678
- C306: LCSC (none) -> C1779
- D301: LCSC (none) -> C134421
- D302, D303: LCSC (none) -> C2297
- FB301: value 600R@100MHz 1A -> 220R@100MHz 2A; LCSC (none) -> C85840; MPN (none) -> BLM21PG221SN1D
- R301: LCSC (none) -> C17477
- R302, R304, R305: LCSC (none) -> C17513
- R303: LCSC (none) -> C17520
- R306, R307: LCSC (none) -> C17798
- U301: LCSC (none) -> C7519
- U302: LCSC (none) -> C8690
Other:
- note added: "Экран J301 не соединять с GND напрямую: R301 0 Ом (DC) и/или C301 (ВЧ), подбор при EMC-испытаниях [AN146 §2.2.2]. C301 4.7n 50 В X7R (DNP) - оценка: AN146 §2.2.2 номинал не задаёт."
- note removed: "Экран J301 не соединять с GND напрямую: R301 0 Ом (DC) и/или C301 (ВЧ), подбор при EMC-испытаниях [AN146 §2.2.2]."
Changed lines of the file:
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@@
 		)
 	)
-	(text "Экран J301 не соединять с GND напрямую: R301 0 Ом (DC)\nи/или C301 (ВЧ), подбор при EMC-испытаниях [AN146 §2.2.2]."
+	(text "Экран J301 не соединять с GND напрямую: R301 0 Ом (DC)\nи/или C301 (ВЧ), подбор при EMC-испытаниях [AN146 §2.2.2].\nC301 4.7n 50 В X7R (DNP) - оценка: AN146 §2.2.2 номинал не задаёт."
 		(exclude_from_sim no)
 		(at 17.78 113.03 0)
@@
 			)
 		)
+		(property "LCSC" "C134421"
+			(at 99.06 30.48 0)
+			(hide yes)
+			(show_name no)
+			(do_not_autoplace no)
+			(effects
+				(font
+					(size 1.27 1.27)
+				)
+			)
+		)
 		(pin "1"
 		)
@@
 			)
 		)
+		(property "LCSC" "C17798"
+			(at 209.55 81.28 0)
+			(hide yes)
+			(show_name no)
+			(do_not_autoplace no)
+			(effects
+				(font
+					(size 1.27 1.27)
+				)
+			)
+		)
 		(pin "1"
 		)
@@
 			)
 		)
+		(property "LCSC" "C17798"
+			(at 209.55 73.66 0)
+			(hide yes)
+			(show_name no)
+			(do_not_autoplace no)
+			(effects
+				(font
+					(size 1.27 1.27)
+				)
+			)
+		)
 		(pin "1"
 		)
@@
 			)
 		)
+		(property "LCSC" "C49678"
+			(at 167.64 36.83 0)
+			(hide yes)
+			(show_name no)
+			(do_not_autoplace no)
+			(effects
+				(font
+					(size 1.27 1.27)
+				)
+			)
+		)
 		(pin "1"
 		)
@@
 			)
 		)
+		(property "LCSC" "C1710"
+			(at 63.5 34.29 0)
+			(hide yes)
+			(show_name no)
+			(do_not_autoplace no)
+			(effects
+				(font
+					(size 1.27 1.27)
+				)
+			)
+		)
 		(pin "1"
 		)
@@
 			)
 		)
+		(property "LCSC" ""
+			(at 30.48 50.8 0)
+			(hide yes)
+			(show_name no)
+			(do_not_autoplace no)
+			(effects
+				(font
+					(size 1.27 1.27)
+				)
+			)
+		)
 		(pin "1"
 		)
@@
 			)
 		)
+		(property "LCSC" "C2297"
+			(at 198.12 81.28 0)
+			(hide yes)
+			(show_name no)
+			(do_not_autoplace no)
+			(effects
+				(font
+					(size 1.27 1.27)
+				)
+			)
+		)
 		(pin "1"
 		)
@@
 			)
 		)
+		(property "LCSC" "C1779"
+			(at 177.8 36.83 0)
+			(hide yes)
+			(show_name no)
+			(do_not_autoplace no)
+			(effects
+				(font
+					(size 1.27 1.27)
+				)
+			)
+		)
 		(pin "1"
 		)
@@
 			)
 		)
+		(property "LCSC" "C17513"
+			(at 190.5 48.26 0)
+			(hide yes)
+			(show_name no)
+			(do_not_autoplace no)
+			(effects
+				(font
+					(size 1.27 1.27)
+				)
+			)
+		)
 		(pin "1"
 		)
@@
 			)
 		)
+		(property "LCSC" "C17513"
+			(at 76.2 34.29 0)
+			(hide yes)
+			(show_name no)
+			(do_not_autoplace no)
+			(effects
+				(font
+					(size 1.27 1.27)
+				)
+			)
+		)
 		(pin "1"
 		)
@@
 			)
 		)
+		(property "LCSC" "C7519"
+			(at 55.88 50.8 0)
+			(hide yes)
+			(show_name no)
+			(do_not_autoplace no)
+			(effects
+				(font
+					(size 1.27 1.27)
+				)
+			)
+		)
 		(pin "1"
 		)
@@
 			)
 		)
+		(property "LCSC" "C17520"
+			(at 76.2 46.99 0)
+			(hide yes)
+			(show_name no)
+			(do_not_autoplace no)
+			(effects
+				(font
+					(size 1.27 1.27)
+				)
+			)
+		)
 		(pin "1"
 		)
@@
 			)
 		)
+		(property "LCSC" "C2297"
+			(at 198.12 73.66 0)
+			(hide yes)
+			(show_name no)
+			(do_not_autoplace no)
+			(effects
+				(font
+					(size 1.27 1.27)
+				)
+			)
+		)
 		(pin "1"
 		)
@@
 			)
 		)
-		(property "Value" "600R@100MHz 1A"
+		(property "Value" "220R@100MHz 2A"
 			(at 87.63 25.4 90)
 			(show_name no)
@@
 			)
 		)
-		(property "Description" "Ferrite bead 0805, >=1 A, 220..600 Ohm @100 MHz"
+		(property "Description" "Ферритовая бусина 220 Ом @100 МГц, 2 А, Rdc 45 мОм, 0805 (Murata BLM21PG221SN1D)"
+			(at 87.63 30.48 0)
+			(hide yes)
+			(show_name no)
+			(do_not_autoplace no)
+			(effects
+				(font
+					(size 1.27 1.27)
+				)
+			)
+		)
+		(property "MPN" "BLM21PG221SN1D"
+			(at 87.63 30.48 0)
+			(hide yes)
+			(show_name no)
+			(do_not_autoplace no)
+			(effects
+				(font
+					(size 1.27 1.27)
+				)
+			)
+		)
+		(property "LCSC" "C85840"
 			(at 87.63 30.48 0)
 			(hide yes)
@@
 			)
 		)
+		(property "LCSC" "C49678"
+			(at 116.84 57.15 0)
+			(hide yes)
+			(show_name no)
+			(do_not_autoplace no)
+			(effects
+				(font
+					(size 1.27 1.27)
+				)
+			)
+		)
 		(pin "1"
 		)
@@
 			)
 		)
+		(property "LCSC" "C49678"
+			(at 147.32 36.83 0)
+			(hide yes)
+			(show_name no)
+			(do_not_autoplace no)
+			(effects
+				(font
+					(size 1.27 1.27)
+				)
+			)
+		)
 		(pin "1"
 		)
@@
 			)
 		)
-		(property "Value" "DNP"
+		(property "Value" "4.7n"
 			(at 36.068 73.66 0)
 			(show_name no)
@@
 			)
 		)
+		(property "LCSC" "C1744"
+			(at 33.02 72.39 0)
+			(hide yes)
+			(show_name no)
+			(do_not_autoplace no)
+			(effects
+				(font
+					(size 1.27 1.27)
+				)
+			)
+		)
 		(pin "1"
 		)
@@
 			)
 		)
+		(property "LCSC" "C17477"
+			(at 22.86 72.39 0)
+			(hide yes)
+			(show_name no)
+			(do_not_autoplace no)
+			(effects
+				(font
+					(size 1.27 1.27)
+				)
+			)
+		)
 		(pin "1"
 		)
@@
 			)
 		)
+		(property "LCSC" "C17513"
+			(at 190.5 55.88 0)
+			(hide yes)
+			(show_name no)
+			(do_not_autoplace no)
+			(effects
+				(font
+					(size 1.27 1.27)
+				)
+			)
+		)
 		(pin "1"
 		)
@@
 			(at 157.48 71.12 0)
 			(hide yes)
+			(show_name no)
+			(do_not_autoplace no)
+			(effects
+				(font
+					(size 1.27 1.27)
+				)
+			)
+		)
+		(property "LCSC" "C8690"
+			(at 157.48 71.12 0)
+			(hide yes)

Commit message: feat(pcb): prepare board for placement
- Зелёные LED остаются C2297 (InGaN), резисторы к ним 330 Ом (C17630):
  ток 0.6-2.1 мА при Vf 2.6-3.1 В. Жёлто-зелёные отклонены: по
  даташитам световая отдача на мА у них в ~10 раз ниже.
- Цепи дифпар переименованы, чтобы KiCad распознавал пары:
  J201_D+/-, STL_D+/-, FT_D+/-, RXI_P/N; шаблоны классов USB90/MDI100
  обновлены.
- Отверстия шилда H801-H804: footprint из шаблона Arduino (NPTH 3.2,
  courtyard 3.4) в проектной библиотеке g0_dev_board.pretty вместо M3
  с courtyard 6.9, конфликтовавшего с разъёмами Uno.
- Исправлена арифметика в комментарии к двухцветному LED ST-Link.
- Плата синхронизирована со схемой: паритет 0, нарушений DRC 0.
Parts:
- R306, R307: value 680 -> 330; LCSC C17798 -> C17630
Connections:
- net USB_DM renamed FT_D-
- net USB_DP renamed FT_D+
Other:
- note added: "CBUS0 = TXLED#, CBUS1 = RXLED# - заводские значения EEPROM [DS табл. 3.4, §7.5 Fig 7.5]. Аноды через 330 Ом (R306/R307) к VCCIO (+3.3V). D302/D303 KT-0805G (C2297, InGaN), Vf 2.6..3.1 В: I = (3.3 - Vf - Vol)/330; без учёта Vol 0.6..2.1 мА; Vol <= 0.5 В при 2 мА [DS табл. 5.4] - при Vf у верхней границы ток мал, яркость проверить на образце."
- note removed: "CBUS0 = TXLED#, CBUS1 = RXLED# - заводские значения EEPROM [DS табл. 3.4, §7.5 Fig 7.5]. Аноды через 680 Ом к VCCIO (+3.3V): I ~ (3.3 - Vf 2.0 - Vol 0.4)/680 ~ 1.3 мА; Vol <= 0.5 В при 2 мА [DS табл. 5.4]. Vf зависит от цвета LED - уточнить."
Changed lines of the file:
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@@
 		)
 	)
-	(text "J301, питание VBUS_FT (вариант A, плата self-powered от +5V):\n- U301 USBLC6-2SC6 первым у разъёма: 1,6 = I/O1 (D+), 3,4 = I/O2 (D-),\n  5 = VBUS, 2 = GND [ULC стр.1; AN146 §2.2.1]. Выводы 1 и 6 (3 и 4)\n  на плате соединить: обе пары в одной цепи.\n- C302 10н и FB301 у разъёма [AN146 §2.4.4 Fig 2.5; DS Fig 6.1].\n- D301 Шоттки VBUS_FT -> +5V: нет обратной подачи с +5V (J201) в VBUS\n  хоста [AN146 §2.4.1]. Такой же диод стоит у J201 (лист st_link).\n- D+/D- напрямую на FT232: внутр. последовательные R и 1.5к на USBDP\n  [DS табл. 3.1]; ферриты на D+/D- запрещены [AN146 §2.4.4]."
+	(text "J301, питание VBUS_FT (вариант A, плата self-powered от +5V):\n- U301 USBLC6-2SC6 первым у разъёма: 1,6 = I/O1 (D+), 3,4 = I/O2 (D-),\n  5 = VBUS, 2 = GND [ULC стр.1; AN146 §2.2.1]. Выводы 1 и 6 (3 и 4)\n  на плате соединить: обе пары в одной цепи.\n- C302 10н и FB301 у разъёма [AN146 §2.4.4 Fig 2.5; DS Fig 6.1].\n- D301 Шоттки VBUS_FT -> +5V: нет обратной подачи с +5V (J201) в VBUS\n  хоста [AN146 §2.4.1]. Такой же диод стоит у J201 (лист st_link).\n- D+/D- (цепи FT_D+/FT_D-; суффиксы +/- - дифпара для KiCad)\n  напрямую на FT232: внутр. последовательные R и 1.5к на USBDP\n  [DS табл. 3.1]; ферриты на D+/D- запрещены [AN146 §2.4.4]."
 		(exclude_from_sim no)
 		(at 17.78 84.455 0)
@@
 		)
 	)
-	(text "CBUS0 = TXLED#, CBUS1 = RXLED# - заводские значения EEPROM\n[DS табл. 3.4, §7.5 Fig 7.5]. Аноды через 680 Ом к VCCIO (+3.3V):\nI ~ (3.3 - Vf 2.0 - Vol 0.4)/680 ~ 1.3 мА; Vol <= 0.5 В при 2 мА\n[DS табл. 5.4]. Vf зависит от цвета LED - уточнить."
+	(text "CBUS0 = TXLED#, CBUS1 = RXLED# - заводские значения EEPROM\n[DS табл. 3.4, §7.5 Fig 7.5]. Аноды через 330 Ом (R306/R307) к VCCIO (+3.3V).\nD302/D303 KT-0805G (C2297, InGaN), Vf 2.6..3.1 В:\nI = (3.3 - Vf - Vol)/330; без учёта Vol 0.6..2.1 мА; Vol <= 0.5 В при 2 мА\n[DS табл. 5.4] - при Vf у верхней границы ток мал, яркость проверить на образце."
 		(exclude_from_sim no)
 		(at 190.5 92.71 0)
@@
 		)
 	)
-	(label "USB_DM"
+	(label "FT_D-"
 		(at 39.37 53.34 0)
 		(effects
@@
 		)
 	)
-	(label "USB_DP"
+	(label "FT_D+"
 		(at 66.04 50.8 0)
 		(effects
@@
 		)
 	)
-	(label "USB_DM"
+	(label "FT_D-"
 		(at 66.04 53.34 0)
 		(effects
@@
 		)
 	)
-	(label "USB_DP"
+	(label "FT_D+"
 		(at 39.37 50.8 0)
 		(effects
@@
 		)
 	)
-	(label "USB_DM"
+	(label "FT_D-"
 		(at 132.08 63.5 180)
 		(effects
@@
 		)
 	)
-	(label "USB_DP"
+	(label "FT_D+"
 		(at 132.08 60.96 180)
 		(effects
@@
 			)
 		)
-		(property "Value" "680"
+		(property "Value" "330"
 			(at 209.55 87.21 90)
 			(show_name no)
@@
 			)
 		)
-		(property "LCSC" "C17798"
+		(property "LCSC" "C17630"
 			(at 209.55 81.28 0)
 			(hide yes)
@@
 			)
 		)
-		(property "Value" "680"
+		(property "Value" "330"
 			(at 209.55 70.27 90)
 			(show_name no)
@@
 			)
 		)
-		(property "LCSC" "C17798"
+		(property "LCSC" "C17630"
 			(at 209.55 73.66 0)
 			(hide yes)
