File: scheme/st_link.kicad_sch (KiCad schematic)
At the start: 41 parts, among them J1 USB_B_Mini, J2 Conn_01x04_Pin, Q1 SS9013, U1 STM32F103CBTx, U5 AP2112K-3.3, Y1 Crystal

Commit message: feat(schematic): fix peripheral sheets and integrate STM32G0B1CCT6
Главный МК заменён на STM32G0B1CCT6 (LQFP-48, pin-to-pin совместим
с STM32G071CBT6). Лист cpu переписан: обвязка по DS13560, LSE
32.768 кГц, подстроечник на ADC (PA4), перемычка JP_IDD, таблица
назначения выводов.

Исправлены листы периферии:
- st_link: перепутанные USB D+/D-, закороченные резисторы SWD,
  VBUS через PTC и Шоттки, ESD USBLC6-2SC6, LDO AP7361C-33E,
  SWO стянут на землю, J2 1x5 с NRST, перемычка JP_STL_PWR;
- ft232rl: 3V3OUT отвязан от общей шины +3.3V, разделены цепи
  TX/RX и светодиодов, ESD, Шоттки на VBUS, делитель на RESET#;
- w5500: номиналы терминации MDI (49.9 Ом / 10 Ом), PMODE=111,
  RSVD на GND, бусина аналогового питания, подтяжки RST/SCS/INT;
- w32: флэш W25Q32JVSSIQ, символ microSD с детектом карты,
  подтяжки линий SD;
- tmp10x: подтяжки I2C, адреса без резисторов, развязка 100 нФ.

Добавлен лист headers: разъёмы Arduino Uno R3 без ICSP, гребёнки
логического анализатора 1x27 с двух сторон, перемычки JP_SWD.
Удалён пустой лист memory. ERC: 0 ошибок.
Parts:
- removed R18: 10k, symbol Device:R
- removed R22: 22, symbol Device:R
- added C110: 10u, Capacitor_SMD:C_0805_2012Metric, symbol Device:C
- added C111: 100n, Capacitor_SMD:C_0805_2012Metric, symbol Device:C
- added C112: 4.7u, Capacitor_SMD:C_0805_2012Metric, symbol Device:C
- added D110: B120, Diode_SMD:D_SMA, symbol Device:D_Schottky
- added F110: MF-MSMF050, Fuse:Fuse_1812_4532Metric, symbol Device:Polyfuse
- added JP202: JP_STL_PWR, Connector_PinHeader_2.54mm:PinHeader_1x02_P2.54mm_Vertical, symbol Connector_Generic:Conn_01x02
- added R110: 0, Resistor_SMD:R_0805_2012Metric, symbol Device:R
- added R111: 100k, Resistor_SMD:R_0805_2012Metric, symbol Device:R
- added U110: USBLC6-2SC6, Package_TO_SOT_SMD:SOT-23-6, symbol Power_Protection:USBLC6-2SC6
- C1: value 1u -> 4.7u; footprint (none) -> Capacitor_SMD:C_0805_2012Metric
- C10, C6, C7, C8, C9: footprint (none) -> Capacitor_SMD:C_0805_2012Metric
- C12, C13: value 20p -> 22p; footprint (none) -> Capacitor_SMD:C_0805_2012Metric
- C4: value 1u -> 10u; footprint (none) -> Capacitor_SMD:C_0805_2012Metric
- D1: value LED -> LED_Green; footprint (none) -> LED_SMD:LED_0805_2012Metric
- D2: value LED -> LED_Red; footprint (none) -> LED_SMD:LED_0805_2012Metric
- D3: footprint (none) -> LED_SMD:LED_0805_2012Metric
- J2: value Conn_01x04_Pin -> F103_SWD; footprint Connector_PinHeader_2.54mm:PinHeader_1x04_P2.54mm_Vertical -> Connector_PinHeader_2.54mm:PinHeader_1x05_P2.54mm_Vertical; symbol Connector:Conn_01x04_Pin -> Connector:Conn_01x05_Pin
- R1, R11, R12, R13, R14, R15, R16, R17, R19, R2, R20, R21, R23, R3, R4, R5, R6, R7, R8: footprint (none) -> Resistor_SMD:R_0805_2012Metric
- R10, R9: value 100 -> 330; footprint (none) -> Resistor_SMD:R_0805_2012Metric
- U1: MPN (none) -> STM32F103CBT6
- U5: value AP2112K-3.3 -> AP7361C-33E; footprint Package_TO_SOT_SMD:SOT-23-5 -> Package_TO_SOT_SMD:SOT-223-3_TabPin2; symbol Regulator_Linear:AP2112K-3.3 -> Regulator_Linear:AP7361C-33E; MPN (none) -> AP7361C-33E-13
- Y1: value Crystal -> 8MHz
Connections:
- net +3.3V: now also U5.3 (VO), JP202.1 (Pin_1); no longer C6.1, C7.1, C8.1, C9.1, D2.2 (A), J2.1 (Pin_1), Q1.3 (C), R12.1, R16.1, U1.24 (VDD), U1.36 (VDD), U1.48 (VDD), U1.9 (VDDA), U5.5 (VOUT)
- net +5V: now also C110.1, C111.1, D110.1 (K); no longer J1.1 (VBUS), R6.1, U5.3 (EN)
- net GND: now also C12.2, C13.2, J2.5 (Pin_5), C110.2, C111.2, C112.2, R111.2, U110.2 (GND); no longer C12.1, C13.1, J2.4 (Pin_4)
- net OSC_IN: now also C12.1, Y1.1; no longer C12.2, Y1.2
- net OSC_OUT: now also C13.1, Y1.2; no longer C13.2, Y1.1
- net RESET: no longer R23.1, U1.18 (PB0)
- net SWCLK: no longer R21.1, U1.15 (PA5), U1.26 (PB13)
- net SWDIO: no longer R19.1, R20.1, U1.25 (PB12)
- net USB_DM: now also R3.2; no longer R2.2
- net USB_DP: now also R2.2; no longer R3.2
- net DM_J1: now reaches J1.2 (D-), R3.1
- net DM_J1: now also U110.3 (I/O2), U110.4 (I/O2)
- net DP_J1: now reaches J1.3 (D+), R2.1
- net DP_J1: now also R1.2, U110.1 (I/O1), U110.6 (I/O1); no longer R1.1
- net STL_SWDIO: now reaches R19.2, U1.27 (PB14)
- net STL_SWDIO: now also R20.1
- net at Q1.1 (E): now also R1.1; no longer R1.2
- net +3V3_STL: now reaches U1.1 (VBAT)
- net +3V3_STL: now also C6.1, C7.1, C8.1, C9.1, D2.2 (A), J2.1 (Pin_1), Q1.3 (C), R12.1, R16.1, U1.24 (VDD), U1.36 (VDD), U1.48 (VDD), U1.9 (VDDA), C112.1, JP202.2 (Pin_2)
- net PA0 renamed T_VCC
- net PC14: no longer names the net of U1.3 (PC14)
- net RST renamed F103_NRST
- net F103_NRST: now also J2.4 (Pin_4)
- net SWCLK_IN renamed F103_SWCLK
- net SWDIO_IN renamed F103_SWDIO
- net SWO renamed STL_SWO_IN
- net STL_SWO_IN: now also R111.1
- new net: D110.2 (A), F110.2
- new net STL_NRST: R23.1, U1.18 (PB0)
- new net STL_PA5: R110.1, U1.15 (PA5)
- new net STL_SWCLK: R110.2, R21.1, U1.26 (PB13)
- new net STL_SWDIO_IN: R19.1, U1.25 (PB12)
- new net VBUS_STL: F110.1, J1.1 (VBUS), R6.1, U110.5 (VBUS)
Other:
- note added: "F103: C6..C9 100n - по одному на VDD 24/36/48 и VDDA 9, C112 4.7u общий на VDD [F103DS рис. 14 Power supply scheme]. VBAT (1) на +3V3_STL (через JP202): батареи нет [MB1136 лист 4; F103DS §2.3.9]."
- note added: "J2 - SWD самого F103 (заливка DAPLink/BMP): 1 = 3V3, 2 = SWDIO (PA13), 3 = SWCLK (PA14), 4 = NRST F103 (connect under reset), 5 = GND."
- note added: "JP202 = JP_STL_PWR: +3.3V (выход U5) -> +3V3_STL - всё питание домена F103: VDD 24/36/48, VDDA 9, VBAT 1, C6..C9, C112, подтяжка NRST R16, LED_STLINK (D2 через PA9), коллектор Q1 (подтяжка D+ 1k5), делитель T_VCC R12/R13, J2 (SWD самого F103). Снять JP202 = выключить программатор: F103 без питания, USB J1 не энумерируется (нет 1k5 на D+). F103 не держит линии SWD; вместе со снятыми JP_SWD (лист h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"
- note added: "LED_STLINK (PA9), двухцветная схема как LD1 в [MB1184]: R9/R10 330R [MB1184 лист 2]. PA9 = 1 -> горит D1, PA9 = 0 -> горит D2. PA9 в Z: цепь +3.3V-D2-R9-R10-D1-GND, сумма Vf красный ~1.8 + зелёный ~2.0 = 3.8 В > 3.3 В -> оба гаснут. Не использовать пару с суммой Vf < 3.3 В (два красных/ИК). Vf уточнить по выбранным LED. R8 0R в катоде D1 - как в [MB1184]."
- note added: "NRST F103: R16 100k + C10 100n [MB1136]. BOOT0 (44) и PB2/BOOT1 (20) - 100k на GND: старт из флэш; для загрузчика ROM - BOOT0 к 3.3 В вручную (BOOT1 = 0 достаточно). PC13 - 10k на GND [MB1136]: BMP читает PC13 как признак ревизии (0 -> не V1) [BMP stlink_common.c]. PC14 - NC: у ST резистор на PC14 не устанавливается [MB1136]; R18 удалён."
- note added: "U5: AP7361C-33E (SOT-223, 1 А) вместо AP2112K-3.3 (SOT-23-5, 600 мА). Бюджет +3.3V: W5500 132 мА + F103 <= 50 + G0B1 + флэш + SD до 100 + LED = 230..340 мА. Vin = +5V - Vf(D110) ~ 4.6 В -> P = (4.6 - 3.3) x I = 0.30..0.44 Вт. AP2112K: θJA 184 °C/W [AP2112 DS] -> ΔT 55..81 °C, Tj до ~106 °C (Ta 25). AP7361C SOT-223: θJA 110 °C/W на мин. площадке [AP7361C DS, Thermal] -> ΔT 33..49 °C; полигон под т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"
- note added: "U5: расчёт замены LDO - в правой колонке листа."
- note added: "USB J1 (ST-LINK): - D+ (J1.3) -> R2 0R -> PA12 (USB_DP); D- (J1.2) -> R3 0R -> PA11 (USB_DM) [F103DS табл. 5: PA11 = USBDM, PA12 = USBDP]. В прежней версии D+/D- были перепутаны. - U110 USBLC6-2SC6 первым у разъёма: 1,6 = I/O1 (D+), 3,4 = I/O2 (D-), 5 = VBUS, 2 = GND [USBLC6-2 DS стр. 1], так же как U30 у J3 (лист ft232rl). 1-6 и 3-4 - одна цепь (метки DP_J1/DM_J1). - Renumeration как в [MB1136 л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"
- note added: "Y1 8 МГц HC49. F103DS табл. 22: CL1 = CL2 5..25 пФ, Cstray (выводы + плата) ~10 пФ. Для кварца с CL = 18 пФ: C = 2 x (CL - Cstray) = 16 пФ при Cstray 10 пФ, 26 пФ при 5 пФ. Выбрано 22 пФ C0G: внутри диапазона F103DS (27 пФ выходит за 25 пФ), эффективная CL = 11 + (5..10) = 16..21 пФ вокруг 18 пФ. Уточнить по CL выбранного кварца. USB FS: допуск 0.25 %, расстройка от CL - десятки ppm."
- note added: "Линии к цели (STM32G0B1, только SWD; SWO у Cortex-M0+ нет): - PB13 SWCLK -> R21 22R -> SWCLK; PB14 SWDIO -> R20 22R -> SWDIO; PB0 NRST -> R23 22R -> RESET [MB1136 лист 4: R5, R8, R13 = 22R]. Выводы - [DAPLINK IO_Config.h, docs/hic/stm32f103xb.md]. - PB12 (вход SWDIO) -> R19 100R -> узел PB14 до 22R [MB1136 R24 100R; MB1184 R80]. DAPLink читает SWDIO только через PB12 (SWDIO_IN_PIN) - без R19 чтен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"
- note added: "Прошивка: DAPLink (HIC stm32f103xb, Apache-2.0) или Black Magic Probe. Штатная прошивка ST на чистый F103 не ставится (нужен загрузчик ST). Неиспользуемые выводы F103 - NC (флаги). У DAPLink PA1 (RTS), PA2 (TX), PB6, PB15 - выходы, PA3 - вход с подтяжкой [DAPLINK uart.c, gpio.c]; у BMP PA6, PA7, PA8 [BMP platform.h, stlink_common.c]. PA2/PA3 (VCP DAPLink, USART2) не выведены: VCP на плате делает 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"
- moved on the sheet: C1, C10, C12, C13, C4, C6, C7, C8, C9, D1, D2, D3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

Commit message: refactor(schematic): re-annotate references by sheet number
Позиционные обозначения перенумерованы по схеме «номер листа x 100»:
cpu - 1xx, st_link - 2xx, ft232rl - 3xx, w5500 - 4xx, w32 - 5xx,
tmp10x - 6xx, leds - 7xx, headers - 8xx. По обозначению на плате
сразу видно, к какому листу относится компонент.

Ссылки на компоненты в текстовых комментариях обновлены. Обозначения
из сторонних референсных схем (MB1136, MB1184, W5500-Ref, Ethernet
Shield, Adafruit) и имена выводов Arduino оставлены без изменений.

Проверено: нетлист до и после совпадает с точностью до переименования
(190 цепей, 187 компонентов), дубликатов нет, ERC - 0 ошибок.
Parts:
- renumbered C6 to C201, C7 to C202, C1 to C203, C8 to C204, C9 to C205, C112 to C206, C4 to C207, C12 to C208, C10 to C209, C110 to C210, C13 to C211, C111 to C212, D2 to D201, D1 to D202, D3 to D203, D110 to D204, F110 to F201, J1 to J201, J2 to J202, JP202 to JP201, Q1 to Q201, R9 to R201, R10 to R202, R11 to R203, R12 to R204, R14 to R205, R15 to R206, R17 to R207, R111 to R208, R4 to R209, R13 to R210, R8 to R211, R1 to R212, R2 to R213, R3 to R214, R16 to R215, R6 to R216, R5 to R217, R7 to R218, R20 to R219, R21 to R220, R23 to R221, R19 to R222, R110 to R223, U110 to U201, U5 to U202, U1 to U203, Y1 to Y201
Other:
- note added: "F103: C201..C205 100n - по одному на VDD 24/36/48 и VDDA 9, C206 4.7u общий на VDD [F103DS рис. 14 Power supply scheme]. VBAT (1) на +3V3_STL (через JP201): батареи нет [MB1136 лист 4; F103DS §2.3.9]."
- note added: "J202 - SWD самого F103 (заливка DAPLink/BMP): 1 = 3V3, 2 = SWDIO (PA13), 3 = SWCLK (PA14), 4 = NRST F103 (connect under reset), 5 = GND."
- note added: "JP201 = JP_STL_PWR: +3.3V (выход U202) -> +3V3_STL - всё питание домена F103: VDD 24/36/48, VDDA 9, VBAT 1, C201..C205, C206, подтяжка NRST R215, LED_STLINK (D201 через PA9), коллектор Q201 (подтяжка D+ 1k5), делитель T_VCC R204/R210, J202 (SWD самого F103). Снять JP201 = выключить программатор: F103 без питания, USB J201 не энумерируется (нет 1k5 на D+). F103 не держит линии SWD; вместе со сняты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"
- note added: "LED_STLINK (PA9), двухцветная схема как LD1 в [MB1184]: R201/R202 330R [MB1184 лист 2]. PA9 = 1 -> горит D202, PA9 = 0 -> горит D201. PA9 в Z: цепь +3.3V-D201-R201-R202-D202-GND, сумма Vf красный ~1.8 + зелёный ~2.0 = 3.8 В > 3.3 В -> оба гаснут. Не использовать пару с суммой Vf < 3.3 В (два красных/ИК). Vf уточнить по выбранным LED. R211 0R в катоде D202 - как в [MB1184]."
- note added: "NRST F103: R215 100k + C209 100n [MB1136]. BOOT0 (44) и PB2/BOOT1 (20) - 100k на GND: старт из флэш; для загрузчика ROM - BOOT0 к 3.3 В вручную (BOOT1 = 0 достаточно). PC13 - 10k на GND [MB1136]: BMP читает PC13 как признак ревизии (0 -> не V1) [BMP stlink_common.c]. PC14 - NC: у ST резистор на PC14 не устанавливается [MB1136]; R18 удалён."
- note added: "U202: AP7361C-33E (SOT-223, 1 А) вместо AP2112K-3.3 (SOT-23-5, 600 мА). Бюджет +3.3V: W5500 132 мА + F103 <= 50 + G0B1 + флэш + SD до 100 + LED = 230..340 мА. Vin = +5V - Vf(D204) ~ 4.6 В -> P = (4.6 - 3.3) x I = 0.30..0.44 Вт. AP2112K: θJA 184 °C/W [AP2112 DS] -> ΔT 55..81 °C, Tj до ~106 °C (Ta 25). AP7361C SOT-223: θJA 110 °C/W на мин. площадке [AP7361C DS, Thermal] -> ΔT 33..49 °C; полигон под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"
- note added: "U202: расчёт замены LDO - в правой колонке листа."
- note added: "USB J201 (ST-LINK): - D+ (J201.3) -> R213 0R -> PA12 (USB_DP); D- (J201.2) -> R214 0R -> PA11 (USB_DM) [F103DS табл. 5: PA11 = USBDM, PA12 = USBDP]. В прежней версии D+/D- были перепутаны. - U201 USBLC6-2SC6 первым у разъёма: 1,6 = I/O1 (D+), 3,4 = I/O2 (D-), 5 = VBUS, 2 = GND [USBLC6-2 DS стр. 1], так же как U301 у J301 (лист ft232rl). 1-6 и 3-4 - одна цепь (метки DP_J1/DM_J1). - Renumeration ка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"
- note added: "Y201 8 МГц HC49. F103DS табл. 22: CL1 = CL2 5..25 пФ, Cstray (выводы + плата) ~10 пФ. Для кварца с CL = 18 пФ: C = 2 x (CL - Cstray) = 16 пФ при Cstray 10 пФ, 26 пФ при 5 пФ. Выбрано 22 пФ C0G: внутри диапазона F103DS (27 пФ выходит за 25 пФ), эффективная CL = 11 + (5..10) = 16..21 пФ вокруг 18 пФ. Уточнить по CL выбранного кварца. USB FS: допуск 0.25 %, расстройка от CL - десятки ppm."
- note added: "Линии к цели (STM32G0B1, только SWD; SWO у Cortex-M0+ нет): - PB13 SWCLK -> R220 22R -> SWCLK; PB14 SWDIO -> R219 22R -> SWDIO; PB0 NRST -> R221 22R -> RESET [MB1136 лист 4: R5, R8, R13 = 22R]. Выводы - [DAPLINK IO_Config.h, docs/hic/stm32f103xb.md]. - PB12 (вход SWDIO) -> R222 100R -> узел PB14 до 22R [MB1136 R24 100R; MB1184 R80]. DAPLink читает SWDIO только через PB12 (SWDIO_IN_PIN) - без R222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"
- note removed: "F103: C6..C9 100n - по одному на VDD 24/36/48 и VDDA 9, C112 4.7u общий на VDD [F103DS рис. 14 Power supply scheme]. VBAT (1) на +3V3_STL (через JP202): батареи нет [MB1136 лист 4; F103DS §2.3.9]."
- note removed: "J2 - SWD самого F103 (заливка DAPLink/BMP): 1 = 3V3, 2 = SWDIO (PA13), 3 = SWCLK (PA14), 4 = NRST F103 (connect under reset), 5 = GND."
- note removed: "JP202 = JP_STL_PWR: +3.3V (выход U5) -> +3V3_STL - всё питание домена F103: VDD 24/36/48, VDDA 9, VBAT 1, C6..C9, C112, подтяжка NRST R16, LED_STLINK (D2 через PA9), коллектор Q1 (подтяжка D+ 1k5), делитель T_VCC R12/R13, J2 (SWD самого F103). Снять JP202 = выключить программатор: F103 без питания, USB J1 не энумерируется (нет 1k5 на D+). F103 не держит линии SWD; вместе со снятыми JP_SWD (лист h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"
- note removed: "LED_STLINK (PA9), двухцветная схема как LD1 в [MB1184]: R9/R10 330R [MB1184 лист 2]. PA9 = 1 -> горит D1, PA9 = 0 -> горит D2. PA9 в Z: цепь +3.3V-D2-R9-R10-D1-GND, сумма Vf красный ~1.8 + зелёный ~2.0 = 3.8 В > 3.3 В -> оба гаснут. Не использовать пару с суммой Vf < 3.3 В (два красных/ИК). Vf уточнить по выбранным LED. R8 0R в катоде D1 - как в [MB1184]."
- note removed: "NRST F103: R16 100k + C10 100n [MB1136]. BOOT0 (44) и PB2/BOOT1 (20) - 100k на GND: старт из флэш; для загрузчика ROM - BOOT0 к 3.3 В вручную (BOOT1 = 0 достаточно). PC13 - 10k на GND [MB1136]: BMP читает PC13 как признак ревизии (0 -> не V1) [BMP stlink_common.c]. PC14 - NC: у ST резистор на PC14 не устанавливается [MB1136]; R18 удалён."
- note removed: "U5: AP7361C-33E (SOT-223, 1 А) вместо AP2112K-3.3 (SOT-23-5, 600 мА). Бюджет +3.3V: W5500 132 мА + F103 <= 50 + G0B1 + флэш + SD до 100 + LED = 230..340 мА. Vin = +5V - Vf(D110) ~ 4.6 В -> P = (4.6 - 3.3) x I = 0.30..0.44 Вт. AP2112K: θJA 184 °C/W [AP2112 DS] -> ΔT 55..81 °C, Tj до ~106 °C (Ta 25). AP7361C SOT-223: θJA 110 °C/W на мин. площадке [AP7361C DS, Thermal] -> ΔT 33..49 °C; полигон под т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"
- note removed: "U5: расчёт замены LDO - в правой колонке листа."
- note removed: "USB J1 (ST-LINK): - D+ (J1.3) -> R2 0R -> PA12 (USB_DP); D- (J1.2) -> R3 0R -> PA11 (USB_DM) [F103DS табл. 5: PA11 = USBDM, PA12 = USBDP]. В прежней версии D+/D- были перепутаны. - U110 USBLC6-2SC6 первым у разъёма: 1,6 = I/O1 (D+), 3,4 = I/O2 (D-), 5 = VBUS, 2 = GND [USBLC6-2 DS стр. 1], так же как U30 у J3 (лист ft232rl). 1-6 и 3-4 - одна цепь (метки DP_J1/DM_J1). - Renumeration как в [MB1136 л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"
- note removed: "Y1 8 МГц HC49. F103DS табл. 22: CL1 = CL2 5..25 пФ, Cstray (выводы + плата) ~10 пФ. Для кварца с CL = 18 пФ: C = 2 x (CL - Cstray) = 16 пФ при Cstray 10 пФ, 26 пФ при 5 пФ. Выбрано 22 пФ C0G: внутри диапазона F103DS (27 пФ выходит за 25 пФ), эффективная CL = 11 + (5..10) = 16..21 пФ вокруг 18 пФ. Уточнить по CL выбранного кварца. USB FS: допуск 0.25 %, расстройка от CL - десятки ppm."
- note removed: "Линии к цели (STM32G0B1, только SWD; SWO у Cortex-M0+ нет): - PB13 SWCLK -> R21 22R -> SWCLK; PB14 SWDIO -> R20 22R -> SWDIO; PB0 NRST -> R23 22R -> RESET [MB1136 лист 4: R5, R8, R13 = 22R]. Выводы - [DAPLINK IO_Config.h, docs/hic/stm32f103xb.md]. - PB12 (вход SWDIO) -> R19 100R -> узел PB14 до 22R [MB1136 R24 100R; MB1184 R80]. DAPLink читает SWDIO только через PB12 (SWDIO_IN_PIN) - без R19 чтен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"

Commit message: fix(schematic): resolve all ERC warnings
ERC: 0 ошибок, 0 предупреждений (было 239 предупреждений).

- w5500, leds: все объекты перенесены на сетку 1.27 мм; удалены
  два провода нулевой длины.
- Заведена проектная библиотека g0_dev_board.kicad_sym (+ sym-lib-table)
  для намеренно изменённых символов: USB_B_Mini с пассивными
  VBUS/GND (J201, J301). Попутно исправлен номер вывода экрана
  6 -> SH: у footprint Lumberg 2486 01 площадки экрана называются SH,
  иначе экран на плате остался бы неподключённым.
- Устаревшие копии символа LED обновлены из стандартной библиотеки.
- Кнопки SW701/SW702: SW_DPST_x2 заменён на SW_Push, footprint
  SW_SPST_PTS645Sx43SMTR92 (площадки 1,1,2,2 уже попарно замкнуты).
- Флэш U501: WP и HOLD подтянуты к +3.3V через R516/R517 10k
  вместо прямого подключения к выходу LDO.

Связность проверена сравнением нетлистов: изменились только цепи
WP/HOLD флэша.
Parts:
- J201: symbol Connector:USB_B_Mini -> g0_dev_board:USB_B_Mini
Connections:
- net GND: now also J201.SH (Shield); no longer J201.6 (Shield)
Changed lines of the file:
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@@
 	)
 	(symbol
-		(lib_id "Connector:USB_B_Mini")
+		(lib_id "g0_dev_board:USB_B_Mini")
 		(at 30.48 55.88 0)
 		(unit 1)
@@
 		(pin "5"
 		)
-		(pin "6"
+		(pin "SH"
 		)
 		(instances

Commit message: fix(schematic): harden FT232 reset and reduce NRST load
- FT232RL: делитель RESET# R302/R303 4.7k/10k -> 1k/2.2k. Обратная
  утечка Шоттки D301 при питании платы от ST-Link поднимала RESET#
  к порогу; теперь порог достигается при 0.59 мА, что выше
  гарантированного IR max B120.
- ST-Link: PTC F201 MF-MSMF050 -> MF-MSMF075 (R1max 1.0 -> 0.45 Ом),
  чтобы VCC FT232 оставался >= 4.0 В в худшем случае.
- NRST: C701 и R703 на листе leds -> DNP. Остаются C103 100n у вывода
  и внутренняя подтяжка, как рекомендует ST (DS13560 рис. 27) и как на
  NUCLEO MB1136.
- SW702: значение RESET -> USER (это пользовательская кнопка на PC13).

Комментарии на схеме обновлены. ERC: 0 ошибок, 0 предупреждений.
Parts:
- F201: value MF-MSMF050 -> MF-MSMF075-2; MPN MF-MSMF050-2 -> MF-MSMF075-2
Changed lines of the file:
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@@
 		)
 	)
-	(text "USB J201 (ST-LINK):\n- D+ (J201.3) -> R213 0R -> PA12 (USB_DP); D- (J201.2) -> R214 0R -> PA11 (USB_DM)\n  [F103DS табл. 5: PA11 = USBDM, PA12 = USBDP]. В прежней версии D+/D- были перепутаны.\n- U201 USBLC6-2SC6 первым у разъёма: 1,6 = I/O1 (D+), 3,4 = I/O2 (D-), 5 = VBUS, 2 = GND\n  [USBLC6-2 DS стр. 1], так же как U301 у J301 (лист ft232rl). 1-6 и 3-4 - одна цепь (метки DP_J1/DM_J1).\n- Renumeration как в [MB1136 лист 4]: Q1 9013, R5 36k / R6 10k, R7 100R, R1 1k5.\n  R212 на D+ со стороны разъёма (до R213). R216 от VBUS_STL (до F201/D204), как от U5V у ST:\n  без кабеля в J201 база Q201 не подтянута даже при питании платы от J301.\n  BMP по высокому уровню на PA15 (10k к VBUS) определяет ревизию V2.1 [BMP stlink_common.c].\n- VBUS: J201 -> VBUS_STL -> F201 MF-MSMF050 (Ihold 0.5 A) -> D204 B120 -> +5V; рядом C210 10u + C212 100n.\n  OR-ing двух USB на диодах, как STPS1L30A в [MB1184 лист 2]; с J301 тот же путь VBUS_FT -> FB301 -> D301.\n  Обратная подача в VBUS хоста недопустима [FTDI AN_146 §2.4.1].\n  Падение до +5V: F201 R1max 1.0 Ом [MF-MSMF DS] + Vf B120 -> при 0.4 А +5V может быть ~4.1..4.4 В.\n  Не проверено: этого хватает для LDO (dropout 0.14 В), но FT232 требует VCC >= 4.0 В [DS_FT232R §6.2]."
+	(text "USB J201 (ST-LINK):\n- D+ (J201.3) -> R213 0R -> PA12 (USB_DP); D- (J201.2) -> R214 0R -> PA11 (USB_DM)\n  [F103DS табл. 5: PA11 = USBDM, PA12 = USBDP]. В прежней версии D+/D- были перепутаны.\n- U201 USBLC6-2SC6 первым у разъёма: 1,6 = I/O1 (D+), 3,4 = I/O2 (D-), 5 = VBUS, 2 = GND\n  [USBLC6-2 DS стр. 1], так же как U301 у J301 (лист ft232rl). 1-6 и 3-4 - одна цепь (метки DP_J1/DM_J1).\n- Renumeration как в [MB1136 лист 4]: Q1 9013, R5 36k / R6 10k, R7 100R, R1 1k5.\n  R212 на D+ со стороны разъёма (до R213). R216 от VBUS_STL (до F201/D204), как от U5V у ST:\n  без кабеля в J201 база Q201 не подтянута даже при питании платы от J301.\n  BMP по высокому уровню на PA15 (10k к VBUS) определяет ревизию V2.1 [BMP stlink_common.c].\n- VBUS: J201 -> VBUS_STL -> F201 MF-MSMF075 (Ihold 0.75 A, R1max 0.45 Ом; MSMF050 с R1max 1.0 Ом\n  давал VCC FT232 < 4.0 В в худшем случае [Bourns MF-MSMF]) -> D204 B120 -> +5V; рядом C210 10u + C212 100n.\n  OR-ing двух USB на диодах, как STPS1L30A в [MB1184 лист 2]; с J301 тот же путь VBUS_FT -> FB301 -> D301.\n  Обратная подача в VBUS хоста недопустима [FTDI AN_146 §2.4.1].\n  Падение до +5V: F201 R1max 1.0 Ом [MF-MSMF DS] + Vf B120 -> при 0.4 А +5V может быть ~4.1..4.4 В.\n  Не проверено: этого хватает для LDO (dropout 0.14 В), но FT232 требует VCC >= 4.0 В [DS_FT232R §6.2]."
 		(exclude_from_sim no)
 		(at 134.62 16.51 0)
@@
 			)
 		)
-		(property "Value" "MF-MSMF050"
+		(property "Value" "MF-MSMF075-2"
 			(at 60.96 24.13 90)
 			(show_name no)
@@
 			)
 		)
-		(property "MPN" "MF-MSMF050-2"
+		(property "MPN" "MF-MSMF075-2"
 			(at 60.96 20.32 0)
 			(hide yes)

Commit message: feat(schematic): add MPN/LCSC fields and fix Q201 pinout
Подготовка к заказу сборки на JLCPCB:
- всем монтируемым символам добавлено скрытое поле LCSC (коды
  проверены через API JLCPCB, по возможности Basic);
- LSE Y101: Epson FC-135 CL 7 пФ (Q13FC13500002), C106/C108 6.8p C0G,
  footprint под ручную пайку; в SDK нужен LSEDRV=10;
- бусины: FB101/FB401 GZ2012D601TF, FB301 BLM21PG221SN1D (2 А);
- Y401 25 МГц X49SD25MSD2SC (CL 20 пФ), C401/C402 27p -> 33p;
- Y201 8 МГц X49SD8MSD2SC, нагрузочные 22p оставлены (предел F103
  25 пФ, сдвиг частоты для USB FS несущественен);
- C505 100n на ~CARD_DET (антидребезг), ссылка на чертёж Hirose.

Исправления:
- Q201: символ SS9013 с распиновкой TO-92 (1=E 2=B 3=C) стоял на
  footprint SOT-23 (1=B 2=E 3=C) - транзистор встал бы неправильно.
  Заменён на MMBT3904 (SOT-23, Basic), цепи B/E/C сохранены;
- лист leds переведён с 1206 на 0805, R701/R702 630 -> 680 Ом
  (630 нет в E24), LD702 ORANGE -> RED;
- C301 (DNP) получил номинал 4.7n, опечатка 25Mhz в Y401.

ERC: 0 ошибок, 0 предупреждений.
Parts:
- C201, C202, C204, C205, C209, C212: LCSC (none) -> C49678
- C203, C206: LCSC (none) -> C1779
- C207, C210: LCSC (none) -> C15850
- C208, C211: LCSC (none) -> C1804
- D201: LCSC (none) -> C84256
- D202, D203: LCSC (none) -> C2297
- D204: LCSC (none) -> C134421
- F201: LCSC (none) -> C84140
- J202: LCSC (none) -> C42431835
- JP201: LCSC (none) -> C42431798
- Q201: value SS9013 -> MMBT3904; footprint Package_TO_SOT_SMD:SOT-23-3 -> Package_TO_SOT_SMD:SOT-23; symbol PCM_Transistor_BJT_AKL:SS9013 -> Transistor_BJT:MMBT3904; LCSC (none) -> C20526
- R201, R202: LCSC (none) -> C17630
- R203: LCSC (none) -> C17513
- R204, R210: LCSC (none) -> C17673
- R205, R206, R208, R209, R215: LCSC (none) -> C149504
- R207, R216: LCSC (none) -> C17414
- R211, R213, R214, R223: LCSC (none) -> C17477
- R212: LCSC (none) -> C4310
- R217: LCSC (none) -> C4360
- R218, R222: LCSC (none) -> C17408
- R219, R220, R221: LCSC (none) -> C17561
- U201: LCSC (none) -> C7519
- U202: LCSC (none) -> C500795
- U203: LCSC (none) -> C8304
- Y201: LCSC (none) -> C21263; MPN (none) -> X49SD8MSD2SC
Connections:
- net at Q201.1 (B): now also R216.2, R217.1, R218.1; no longer R212.1
- new net: Q201.2 (E), R212.1
Other:
- note added: "Y201 8 МГц HC49: YXC X49SD8MSD2SC, CL = 20 пФ, ESR <= 60 Ом [DS YXC HC-49US]. F103DS табл. 22: CL1 = CL2 5..25 пФ, Cstray (выводы + плата) ~5..10 пФ. Под CL = 20 пФ надо C = 2 x (20 - Cstray) = 20..30 пФ, но 33 пФ вне 5..25 пФ F103DS - не ставим. Оставлено 22 пФ C0G: эффективная CL = 11 + (5..10) = 16..21 пФ при номинале кварца 20 пФ. Сдвиг частоты от недогрузки - десятки ppm; для USB FS (допуск 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"
- note removed: "Y201 8 МГц HC49. F103DS табл. 22: CL1 = CL2 5..25 пФ, Cstray (выводы + плата) ~10 пФ. Для кварца с CL = 18 пФ: C = 2 x (CL - Cstray) = 16 пФ при Cstray 10 пФ, 26 пФ при 5 пФ. Выбрано 22 пФ C0G: внутри диапазона F103DS (27 пФ выходит за 25 пФ), эффективная CL = 11 + (5..10) = 16..21 пФ вокруг 18 пФ. Уточнить по CL выбранного кварца. USB FS: допуск 0.25 %, расстройка от CL - десятки ppm."
