File: scheme/st_link.kicad_sch (KiCad schematic)
At the start: 48 parts, among them J201 USB_B_Mini, J202 F103_SWD, Q201 MMBT3904, U201 USBLC6-2SC6, U202 AP7361C-33E, U203 STM32F103CBTx, Y201 8MHz

Commit message: feat(pcb): prepare board for placement
- Зелёные LED остаются C2297 (InGaN), резисторы к ним 330 Ом (C17630):
  ток 0.6-2.1 мА при Vf 2.6-3.1 В. Жёлто-зелёные отклонены: по
  даташитам световая отдача на мА у них в ~10 раз ниже.
- Цепи дифпар переименованы, чтобы KiCad распознавал пары:
  J201_D+/-, STL_D+/-, FT_D+/-, RXI_P/N; шаблоны классов USB90/MDI100
  обновлены.
- Отверстия шилда H801-H804: footprint из шаблона Arduino (NPTH 3.2,
  courtyard 3.4) в проектной библиотеке g0_dev_board.pretty вместо M3
  с courtyard 6.9, конфликтовавшего с разъёмами Uno.
- Исправлена арифметика в комментарии к двухцветному LED ST-Link.
- Плата синхронизирована со схемой: паритет 0, нарушений DRC 0.
Parts:
- R203: value 1k -> 330; LCSC C17513 -> C17630
Connections:
- net DM_J1 renamed J201_D-
- net DP_J1 renamed J201_D+
- net USB_DM renamed STL_D-
- net USB_DP renamed STL_D+
Other:
- note added: "LED_STLINK (PA9), двухцветная схема как LD1 в [MB1184]: R201/R202 330R [MB1184 лист 2]. PA9 = 1 -> горит D202, PA9 = 0 -> горит D201. PA9 в Z: цепь +3.3V-D201-R201-R202-D202-GND, сумма минимальных Vf: D201 NCD0805R1 (C84256, красный) 1.5 В + D202 KT-0805G (C2297, зелёный) 2.6 В @5 мА = 4.1 В > 3.3 В -> оба гаснут [даташиты NCD0805R1, KT-0805G]. Не использовать пару с суммой Vf < 3.3 В (два красны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"
- note added: "USB J201 (ST-LINK): - D+ (J201.3) -> R213 0R -> PA12 (цепь STL_D+); D- (J201.2) -> R214 0R -> PA11 (цепь STL_D-) [F103DS табл. 5: PA11 = USBDM, PA12 = USBDP]. В прежней версии D+/D- были перепутаны. - U201 USBLC6-2SC6 первым у разъёма: 1,6 = I/O1 (D+), 3,4 = I/O2 (D-), 5 = VBUS, 2 = GND [USBLC6-2 DS стр. 1], так же как U301 у J301 (лист ft232rl). 1-6 и 3-4 - одна цепь (метки J201_D+/J201_D-). Суф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"
- note removed: "LED_STLINK (PA9), двухцветная схема как LD1 в [MB1184]: R201/R202 330R [MB1184 лист 2]. PA9 = 1 -> горит D202, PA9 = 0 -> горит D201. PA9 в Z: цепь +3.3V-D201-R201-R202-D202-GND, сумма Vf красный ~1.8 + зелёный ~2.0 = 3.8 В > 3.3 В -> оба гаснут. Не использовать пару с суммой Vf < 3.3 В (два красных/ИК). Vf уточнить по выбранным LED. R211 0R в катоде D202 - как в [MB1184]."
- note removed: "USB J201 (ST-LINK): - D+ (J201.3) -> R213 0R -> PA12 (USB_DP); D- (J201.2) -> R214 0R -> PA11 (USB_DM) [F103DS табл. 5: PA11 = USBDM, PA12 = USBDP]. В прежней версии D+/D- были перепутаны. - U201 USBLC6-2SC6 первым у разъёма: 1,6 = I/O1 (D+), 3,4 = I/O2 (D-), 5 = VBUS, 2 = GND [USBLC6-2 DS стр. 1], так же как U301 у J301 (лист ft232rl). 1-6 и 3-4 - одна цепь (метки DP_J1/DM_J1). - Renumeration ка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"
Changed lines of the file:
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@@
 		)
 	)
-	(text "JP201 = JP_STL_PWR: +3.3V (выход U202) -> +3V3_STL - всё питание домена F103: VDD 24/36/48, VDDA 9,\nVBAT 1, C201..C205, C206, подтяжка NRST R215, LED_STLINK (D201 через PA9), коллектор Q201 (подтяжка D+ 1k5),\nделитель T_VCC R204/R210, J202 (SWD самого F103).\nСнять JP201 = выключить программатор: F103 без питания, USB J201 не энумерируется (нет 1k5 на D+).\nF103 не держит линии SWD; вместе со снятыми JP_SWD (лист headers) - полная изоляция МК.\nДелитель T_VCC и D201 переведены на +3V3_STL, чтобы при снятом JP201 не подпитывать F103 через PA0/PA9.\nD203 (индикатор питания) оставлен на +3.3V - показывает питание платы. U202 и всё остальное - без изменений."
+	(text "JP201 = JP_STL_PWR: +3.3V (выход U202) -> +3V3_STL - всё питание домена F103: VDD 24/36/48, VDDA 9,\nVBAT 1, C201..C205, C206, подтяжка NRST R215, LED_STLINK (D201 через PA9), коллектор Q201 (подтяжка D+ 1k5),\nделитель T_VCC R204/R210, J202 (SWD самого F103).\nСнять JP201 = выключить программатор: F103 без питания, USB J201 не энумерируется (нет 1k5 на D+).\nF103 не держит линии SWD; вместе со снятыми JP_SWD (лист headers) - полная изоляция МК.\nДелитель T_VCC и D201 переведены на +3V3_STL, чтобы при снятом JP201 не подпитывать F103 через PA0/PA9.\nD203 (индикатор питания) оставлен на +3.3V - показывает питание платы. U202 и всё остальное - без изменений.\nD203 KT-0805G (C2297, InGaN, Vf 2.6..3.1 В) + R203 330R: I = (3.3 - Vf)/330 = 0.6..2.1 мА."
 		(exclude_from_sim no)
 		(at 167.64 220.98 0)
@@
 		)
 	)
-	(text "USB J201 (ST-LINK):\n- D+ (J201.3) -> R213 0R -> PA12 (USB_DP); D- (J201.2) -> R214 0R -> PA11 (USB_DM)\n  [F103DS табл. 5: PA11 = USBDM, PA12 = USBDP]. В прежней версии D+/D- были перепутаны.\n- U201 USBLC6-2SC6 первым у разъёма: 1,6 = I/O1 (D+), 3,4 = I/O2 (D-), 5 = VBUS, 2 = GND\n  [USBLC6-2 DS стр. 1], так же как U301 у J301 (лист ft232rl). 1-6 и 3-4 - одна цепь (метки DP_J1/DM_J1).\n- Renumeration как в [MB1136 лист 4]: Q1 9013, R5 36k / R6 10k, R7 100R, R1 1k5.\n  Q201 = MMBT3904 вместо 9013: функционально подходит любой малосигнальный NPN (ST ставит 9013),\n  MMBT3904 - стандартный SOT-23 с однозначной распиновкой 1=B 2=E 3=C, Basic в JLCPCB (C20526).\n  R212 на D+ со стороны разъёма (до R213). R216 от VBUS_STL (до F201/D204), как от U5V у ST:\n  без кабеля в J201 база Q201 не подтянута даже при питании платы от J301.\n  BMP по высокому уровню на PA15 (10k к VBUS) определяет ревизию V2.1 [BMP stlink_common.c].\n- VBUS: J201 -> VBUS_STL -> F201 MF-MSMF075 (Ihold 0.75 A, R1max 0.45 Ом; MSMF050 с R1max 1.0 Ом\n  давал VCC FT232 < 4.0 В в худшем случае [Bourns MF-MSMF]) -> D204 B120 -> +5V; рядом C210 10u + C212 100n.\n  OR-ing двух USB на диодах, как STPS1L30A в [MB1184 лист 2]; с J301 тот же путь VBUS_FT -> FB301 -> D301.\n  Обратная подача в VBUS хоста недопустима [FTDI AN_146 §2.4.1].\n  Падение до +5V: F201 R1max 1.0 Ом [MF-MSMF DS] + Vf B120 -> при 0.4 А +5V может быть ~4.1..4.4 В.\n  Не проверено: этого хватает для LDO (dropout 0.14 В), но FT232 требует VCC >= 4.0 В [DS_FT232R §6.2]."
+	(text "USB J201 (ST-LINK):\n- D+ (J201.3) -> R213 0R -> PA12 (цепь STL_D+); D- (J201.2) -> R214 0R -> PA11 (цепь STL_D-)\n  [F103DS табл. 5: PA11 = USBDM, PA12 = USBDP]. В прежней версии D+/D- были перепутаны.\n- U201 USBLC6-2SC6 первым у разъёма: 1,6 = I/O1 (D+), 3,4 = I/O2 (D-), 5 = VBUS, 2 = GND\n  [USBLC6-2 DS стр. 1], так же как U301 у J301 (лист ft232rl). 1-6 и 3-4 - одна цепь (метки J201_D+/J201_D-).\n  Суффиксы +/- в именах цепей - чтобы KiCad распознал дифпары J201_D+/- и STL_D+/-.\n- Renumeration как в [MB1136 лист 4]: Q1 9013, R5 36k / R6 10k, R7 100R, R1 1k5.\n  Q201 = MMBT3904 вместо 9013: функционально подходит любой малосигнальный NPN (ST ставит 9013),\n  MMBT3904 - стандартный SOT-23 с однозначной распиновкой 1=B 2=E 3=C, Basic в JLCPCB (C20526).\n  R212 на D+ со стороны разъёма (до R213). R216 от VBUS_STL (до F201/D204), как от U5V у ST:\n  без кабеля в J201 база Q201 не подтянута даже при питании платы от J301.\n  BMP по высокому уровню на PA15 (10k к VBUS) определяет ревизию V2.1 [BMP stlink_common.c].\n- VBUS: J201 -> VBUS_STL -> F201 MF-MSMF075 (Ihold 0.75 A, R1max 0.45 Ом; MSMF050 с R1max 1.0 Ом\n  давал VCC FT232 < 4.0 В в худшем случае [Bourns MF-MSMF]) -> D204 B120 -> +5V; рядом C210 10u + C212 100n.\n  OR-ing двух USB на диодах, как STPS1L30A в [MB1184 лист 2]; с J301 тот же путь VBUS_FT -> FB301 -> D301.\n  Обратная подача в VBUS хоста недопустима [FTDI AN_146 §2.4.1].\n  Падение до +5V: F201 R1max 1.0 Ом [MF-MSMF DS] + Vf B120 -> при 0.4 А +5V может быть ~4.1..4.4 В.\n  Не проверено: этого хватает для LDO (dropout 0.14 В), но FT232 требует VCC >= 4.0 В [DS_FT232R §6.2]."
 		(exclude_from_sim no)
 		(at 134.62 16.51 0)
@@
 		)
 	)
-	(text "LED_STLINK (PA9), двухцветная схема как LD1 в [MB1184]: R201/R202 330R [MB1184 лист 2].\nPA9 = 1 -> горит D202, PA9 = 0 -> горит D201. PA9 в Z: цепь +3.3V-D201-R201-R202-D202-GND,\nсумма Vf красный ~1.8 + зелёный ~2.0 = 3.8 В > 3.3 В -> оба гаснут.\nНе использовать пару с суммой Vf < 3.3 В (два красных/ИК). Vf уточнить по выбранным LED.\nR211 0R в катоде D202 - как в [MB1184]."
+	(text "LED_STLINK (PA9), двухцветная схема как LD1 в [MB1184]: R201/R202 330R [MB1184 лист 2].\nPA9 = 1 -> горит D202, PA9 = 0 -> горит D201. PA9 в Z: цепь +3.3V-D201-R201-R202-D202-GND,\nсумма минимальных Vf: D201 NCD0805R1 (C84256, красный) 1.5 В + D202 KT-0805G (C2297, зелёный)\n2.6 В @5 мА = 4.1 В > 3.3 В -> оба гаснут [даташиты NCD0805R1, KT-0805G].\nНе использовать пару с суммой Vf < 3.3 В (два красных/ИК).\nR211 0R в катоде D202 - как в [MB1184]."
 		(exclude_from_sim no)
 		(at 80.01 203.2 0)
@@
 		)
 	)
-	(label "DM_J1"
+	(label "J201_D-"
 		(at 40.64 58.42 0)
 		(effects
@@
 		)
 	)
-	(label "USB_DM"
+	(label "STL_D-"
 		(at 96.52 63.5 0)
 		(effects
@@
 		)
 	)
-	(label "USB_DP"
+	(label "STL_D+"
 		(at 228.6 99.06 0)
 		(effects
@@
 		)
 	)
-	(label "DP_J1"
+	(label "J201_D+"
 		(at 40.64 55.88 0)
 		(effects
@@
 		)
 	)
-	(label "DP_J1"
+	(label "J201_D+"
 		(at 63.5 55.88 0)
 		(effects
@@
 		)
 	)
-	(label "DM_J1"
+	(label "J201_D-"
 		(at 63.5 58.42 0)
 		(effects
@@
 		)
 	)
-	(label "USB_DM"
+	(label "STL_D-"
 		(at 228.6 96.52 0)
 		(effects
@@
 		)
 	)
-	(label "USB_DP"
+	(label "STL_D+"
 		(at 96.52 55.88 0)
 		(effects
@@
 			)
 		)
-		(property "Value" "1k"
+		(property "Value" "330"
 			(at 35.56 170.18 90)
 			(show_name no)
@@
 			)
 		)
-		(property "LCSC" "C17513"
+		(property "LCSC" "C17630"
 			(at 35.56 167.64 0)
 			(hide yes)
