File: scheme/w5500.kicad_sch (KiCad schematic)
At the start: 55 parts, among them J401 RJ45_Hanrun_HR911105A_Horizon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, U401 W5500, Y401 25Mhz

Commit message: feat(schematic): add MPN/LCSC fields and fix Q201 pinout
Подготовка к заказу сборки на JLCPCB:
- всем монтируемым символам добавлено скрытое поле LCSC (коды
  проверены через API JLCPCB, по возможности Basic);
- LSE Y101: Epson FC-135 CL 7 пФ (Q13FC13500002), C106/C108 6.8p C0G,
  footprint под ручную пайку; в SDK нужен LSEDRV=10;
- бусины: FB101/FB401 GZ2012D601TF, FB301 BLM21PG221SN1D (2 А);
- Y401 25 МГц X49SD25MSD2SC (CL 20 пФ), C401/C402 27p -> 33p;
- Y201 8 МГц X49SD8MSD2SC, нагрузочные 22p оставлены (предел F103
  25 пФ, сдвиг частоты для USB FS несущественен);
- C505 100n на ~CARD_DET (антидребезг), ссылка на чертёж Hirose.

Исправления:
- Q201: символ SS9013 с распиновкой TO-92 (1=E 2=B 3=C) стоял на
  footprint SOT-23 (1=B 2=E 3=C) - транзистор встал бы неправильно.
  Заменён на MMBT3904 (SOT-23, Basic), цепи B/E/C сохранены;
- лист leds переведён с 1206 на 0805, R701/R702 630 -> 680 Ом
  (630 нет в E24), LD702 ORANGE -> RED;
- C301 (DNP) получил номинал 4.7n, опечатка 25Mhz в Y401.

ERC: 0 ошибок, 0 предупреждений.
Parts:
- C401, C402: value 27p C0G -> 33p C0G; LCSC (none) -> C157687
- C403, C404, C405, C408, C410, C412, C413: LCSC (none) -> C49678
- C406, C407: LCSC (none) -> C1755
- C409, C414: LCSC (none) -> C15850
- C411: LCSC (none) -> C1729
- C415, C417: LCSC (none) -> C1710
- C416: LCSC (none) -> C1779
- D401, D402, D403, D404: LCSC (none) -> C2297
- FB401: value FB 600R@100MHz 0805 -> 600R@100MHz 0.5A; LCSC (none) -> C1017; MPN (none) -> GZ2012D601TF
- J401: LCSC (none) -> C12074
- R401, R402, R403, R410, R411, R412, R413, R414, R415, R416, R417: LCSC (none) -> C17414
- R404, R405, R406, R407, R408, R409: LCSC (none) -> C17561
- R418: LCSC (none) -> C17514
- R419, R420, R422, R423: LCSC (none) -> C17720
- R421: LCSC (none) -> C17415
- R424, R425, R426, R427: LCSC (none) -> C17513
- R428: LCSC (none) -> C30908
- R429, R430: LCSC (none) -> C17630
- U401: LCSC (none) -> C32843
- Y401: value 25Mhz -> 25MHz; LCSC (none) -> C14730; MPN (none) -> X49SD25MSD2SC
Other:
- note added: "FB401 + 3V3A: AVDD (выв. 4/8/11/15/17/21) и R419–R421 через бусину — W5500-Ref L1, прим. (1)g: 100–2000 Ом @100 МГц. GZ2012D601TF: 600 Ом, 0.5 А. C403–C413, C409 — на 3V3A; C405, C414 — на +3.3V (VDD). AGND = GND (DG стр.3). R428 12k4 1% (E96): задан DS стр.8 (EXRES1 12.4 кОм 1%), в E24 нет."
- note added: "Y401 25 МГц: YXC X49SD25MSD2SC, CL 20 пФ, ESR <= 40 Ом, ±20 ppm [DS YXC]. W5500 DS 5.5.3 стр.60: C0 <= 7 пФ, ±30 ppm. CL 18 пФ в LCSC нет -> CL 20 пФ. C402/C401 = 2·(CL − Cstray) = 2·(20 − ~4) = 32 → 33 пФ (E24), C0G/NP0. WIZnet (DS рис.3, W5500-Ref C13/C14) ставит 18p: CL_eff ≈ 9 + Cstray ≈ 13 пФ. Ethernet ±50 ppm. Cstray (выводы + трассы) — оценка; частоту проверить."
- note removed: "FB401 + 3V3A: AVDD (выв. 4/8/11/15/17/21) и R419–R421 через бусину — W5500-Ref L1, прим. (1)g: 100–2000 Ом @100 МГц. MPN не выбран (ток >= 0.5 А). C403–C413, C409 — на 3V3A; C405, C414 — на +3.3V (VDD). AGND = GND (DG стр.3). R428 12k4 1% (E96): задан DS стр.8 (EXRES1 12.4 кОм 1%), в E24 нет."
- note removed: "Y401 25 МГц: кварц с CL = 18 пФ (DS 5.5.3 стр.60; C0 <= 7 пФ, ±30 ppm). C402/C401 = 2·(CL − Cstray) = 2·(18 − ~4.5) ≈ 27 пФ (E24), C0G/NP0. WIZnet (DS рис.3 стр.11, W5500-Ref C13/C14) ставит 18p: CL_eff ≈ 9 + Cstray ≈ 13 пФ — частота уходит вверх. Cstray (выводы + трассы) — оценка. При кварце с другим CL — пересчитать; частоту проверить на прототипе."

Commit message: feat(pcb): prepare board for placement
- Зелёные LED остаются C2297 (InGaN), резисторы к ним 330 Ом (C17630):
  ток 0.6-2.1 мА при Vf 2.6-3.1 В. Жёлто-зелёные отклонены: по
  даташитам световая отдача на мА у них в ~10 раз ниже.
- Цепи дифпар переименованы, чтобы KiCad распознавал пары:
  J201_D+/-, STL_D+/-, FT_D+/-, RXI_P/N; шаблоны классов USB90/MDI100
  обновлены.
- Отверстия шилда H801-H804: footprint из шаблона Arduino (NPTH 3.2,
  courtyard 3.4) в проектной библиотеке g0_dev_board.pretty вместо M3
  с courtyard 6.9, конфликтовавшего с разъёмами Uno.
- Исправлена арифметика в комментарии к двухцветному LED ST-Link.
- Плата синхронизирована со схемой: паритет 0, нарушений DRC 0.
Parts:
- R424, R425, R426, R427: value 1k -> 330; LCSC C17513 -> C17630
Connections:
- net RXNNET renamed RXI_N
- net RXPNET renamed RXI_P
Other:
- note added: "LED D401–D404: KT-0805G (C2297, InGaN), Vf 2.6–3.1 В; R424–R427 330R: I = (3.3 − Vf)/330 = 0.6–2.1 мА (без Vol). ACTLED/LINKLED: D403/D404 ≤ 2.1 + J401 ≈ 4 < 8 мА (IOL). Имена цепей MDI для дифпар KiCad (суффикс P/N): TXP/TXN, RXP/RXN; со стороны W5500 RXIP/RXIN — цепи RXI_P/RXI_N."
- note added: "R429/R430 330R — как W5500-Ref R8/R9. I ≈ (3.3 − Vf)/330 ≈ 4 мА (Vf ≈ 2 В — оценка, в даташ. HR911105A нет). IOL W5500 8 мА @0.4 В (DS стр.59); с D403/D404 суммарно < 6.1 мА."
- note removed: "R429/R430 330R — как W5500-Ref R8/R9. I ≈ (3.3 − Vf)/330 ≈ 4 мА (Vf ≈ 2 В — оценка, в даташ. HR911105A нет). IOL W5500 8 мА @0.4 В (DS стр.59); с D403/D404 суммарно < 6 мА."
Changed lines of the file:
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@@
 		)
 	)
+	(text "LED D401–D404: KT-0805G (C2297, InGaN), Vf 2.6–3.1 В;\nR424–R427 330R: I = (3.3 − Vf)/330 = 0.6–2.1 мА (без Vol).\nACTLED/LINKLED: D403/D404 ≤ 2.1 + J401 ≈ 4 < 8 мА (IOL).\nИмена цепей MDI для дифпар KiCad (суффикс P/N): TXP/TXN,\nRXP/RXN; со стороны W5500 RXIP/RXIN — цепи RXI_P/RXI_N."
+		(exclude_from_sim no)
+		(at 15.24 104.14 0)
+		(effects
+			(font
+				(size 1.27 1.27)
+			)
+			(justify left top)
+		)
+	)
 	(text "MDI: W5500-Ref (R1/R2/R6/R7 49R9 1%, R3 10R 1%, C9/C10 6n8,\nC8 22n, C15 10n), DG стр.3. 49R9 (E96): 2×49.9 = 100 Ом.\nTXP→TD+ (J401.1), RXP→RD+ (J401.3): как в W5500-Ref (линии\nу R21/R22 перекрещены) и HR911105A (P1 TD+, P3 RD+). DG\nстр.3 — обобщённый рисунок. Auto-MDIX нет (DS 5.5.6)."
 		(exclude_from_sim no)
@@
 		)
 	)
-	(text "R429/R430 330R — как\nW5500-Ref R8/R9.\nI ≈ (3.3 − Vf)/330 ≈ 4 мА\n(Vf ≈ 2 В — оценка, в\nдаташ. HR911105A нет).\nIOL W5500 8 мА @0.4 В\n(DS стр.59); с D403/D404\nсуммарно < 6 мА."
+	(text "R429/R430 330R — как\nW5500-Ref R8/R9.\nI ≈ (3.3 − Vf)/330 ≈ 4 мА\n(Vf ≈ 2 В — оценка, в\nдаташ. HR911105A нет).\nIOL W5500 8 мА @0.4 В\n(DS стр.59); с D403/D404\nсуммарно < 6.1 мА."
 		(exclude_from_sim no)
 		(at 259.08 41.91 0)
@@
 		)
 	)
-	(label "RXNNET"
+	(label "RXI_N"
 		(at 222.25 55.88 0)
 		(effects
@@
 		)
 	)
-	(label "RXPNET"
+	(label "RXI_P"
 		(at 151.13 69.85 180)
 		(effects
@@
 		)
 	)
-	(label "RXPNET"
+	(label "RXI_P"
 		(at 222.25 66.04 0)
 		(effects
@@
 		)
 	)
-	(label "RXPNET"
+	(label "RXI_P"
 		(at 172.72 36.83 0)
 		(effects
@@
 		)
 	)
-	(label "RXNNET"
+	(label "RXI_N"
 		(at 172.72 24.13 0)
 		(effects
@@
 		)
 	)
-	(label "RXNNET"
+	(label "RXI_N"
 		(at 151.13 67.31 180)
 		(effects
@@
 			)
 		)
-		(property "Value" "1k"
+		(property "Value" "330"
 			(at 259.08 89.3195 90)
 			(show_name no)
@@
 			)
 		)
-		(property "LCSC" "C17513"
+		(property "LCSC" "C17630"
 			(at 259.08 92.71 0)
 			(hide yes)
@@
 			)
 		)
-		(property "Value" "1k"
+		(property "Value" "330"
 			(at 259.08 123.6095 90)
 			(show_name no)
@@
 			)
 		)
-		(property "LCSC" "C17513"
+		(property "LCSC" "C17630"
 			(at 259.08 127 0)
 			(hide yes)
@@
 			)
 		)
-		(property "Value" "1k"
+		(property "Value" "330"
 			(at 259.08 99.4795 90)
 			(show_name no)
@@
 			)
 		)
-		(property "LCSC" "C17513"
+		(property "LCSC" "C17630"
 			(at 259.08 102.87 0)
 			(hide yes)
@@
 			)
 		)
-		(property "Value" "1k"
+		(property "Value" "330"
 			(at 259.08 112.1795 90)
 			(show_name no)
@@
 			)
 		)
-		(property "LCSC" "C17513"
+		(property "LCSC" "C17630"
 			(at 259.08 115.57 0)
 			(hide yes)
