File: scheme/headers.kicad_sch (KiCad schematic)
At the start: 12 parts, among them J200 Uno_IOH, J201 Uno_IOL, J202 Uno_POWER, J203 Uno_ANALOG, J204 J_LA_L, J205 J_LA_R

Commit message: refactor(schematic): re-annotate references by sheet number
Позиционные обозначения перенумерованы по схеме «номер листа x 100»:
cpu - 1xx, st_link - 2xx, ft232rl - 3xx, w5500 - 4xx, w32 - 5xx,
tmp10x - 6xx, leds - 7xx, headers - 8xx. По обозначению на плате
сразу видно, к какому листу относится компонент.

Ссылки на компоненты в текстовых комментариях обновлены. Обозначения
из сторонних референсных схем (MB1136, MB1184, W5500-Ref, Ethernet
Shield, Adafruit) и имена выводов Arduino оставлены без изменений.

Проверено: нетлист до и после совпадает с точностью до переименования
(190 цепей, 187 компонентов), дубликатов нет, ERC - 0 ошибок.
Parts:
- renumbered D200 to D801, D201 to D802, J200 to J801, J201 to J802, J202 to J803, J203 to J804, J204 to J805, J205 to J806, JP201 to JP801, R201 to R801, R202 to R802, R203 to R803
Other:
- note added: "AREF: R801 0R DNP на VREF+. VREF+ допустимо от 2 В до VDDA = 3.3 В (DS13560 §3.7.1); перед установкой R801 выпаять FB101 (лист cpu), иначе AREF шилда закорачивается на +3V3_MCU."
- note added: "JP801 = JP_SWD (как CN2 на NUCLEO / CN3 на Discovery): нечётный ряд - ST-LINK (STL_SWCLK, STL_SWDIO, STL_RESET, GND), чётный - МК (PA14, PA13, NRST, GND). Три джампера 1-2, 3-4, 5-6 = программатор подключён к своему МК. Джамперы сняты -> нечётный ряд + GND (выв. 7) = SWD-выход на внешнюю плату (питание цели отдельно, уровни 3.3 В). Выбран 2x4: пара 7-8 (GND-GND) даёт GND рядом с SWD и место для х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"
- note added: "PWR_FLAG: +5V (источники - диоды D204/D301, пассивные) и GND (после смены типа GND у USB_B_Mini на passive)."
- note added: "RESET шилда: D802 BAT54WS, анод - NRST, катод - вывод RESET разъёма. Кнопка шилда тянет RESET к GND -> NRST = Vf ~0.25-0.3 В при токе внутр. подтяжки (~40-80 мкА) < VIL(NRST) (DS13560 табл. 60). 5 В с шилда на RESET запирают диод и в NRST не попадают. Ограничение: шилд не видит сброс платы (вывод RESET разъёма не повторяет уровень NRST)."
- note added: "VIN: D801 B120 от +5V, катод к VIN шилда. Шилд с собственным питанием на VIN (CNC Shield, GSM) не может подать напряжение в +5V платы и в USB-хост (обратный ток блокируется диодом). На VIN платы = +5V - Vf (~0.3-0.5 В). Внешнее питание платы через VIN не предусмотрено."
- note added: "Гребёнки логического анализатора, 1x27 каждая (одинаковые, по левому и правому краю платы, подпись каждого вывода - на шелкографии): J806 J_LA_R (цифровой ряд Uno): SCL, SDA, AREF, GND, D13..D8, D7..D0 (порядок IOH+IOL), GND, SPI2 SCK/MISO/MOSI, W_CS, W_INT, U1_TX, U1_RX, GND. J805 J_LA_L (POWER/ANALOG): GND, 3V3, NRST, 5V, GND, VIN, A0..A5, GND, FL_CS, SD_CS, CARD_DET, W_RST, LED0, LED1, BTN, PO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"
- note removed: "AREF: R201 0R DNP на VREF+. VREF+ допустимо от 2 В до VDDA = 3.3 В (DS13560 §3.7.1); перед установкой R201 выпаять FB200 (лист cpu), иначе AREF шилда закорачивается на +3V3_MCU."
- note removed: "JP201 = JP_SWD (как CN2 на NUCLEO / CN3 на Discovery): нечётный ряд - ST-LINK (STL_SWCLK, STL_SWDIO, STL_RESET, GND), чётный - МК (PA14, PA13, NRST, GND). Три джампера 1-2, 3-4, 5-6 = программатор подключён к своему МК. Джамперы сняты -> нечётный ряд + GND (выв. 7) = SWD-выход на внешнюю плату (питание цели отдельно, уровни 3.3 В). Выбран 2x4: пара 7-8 (GND-GND) даёт GND рядом с SWD и место для х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"
- note removed: "PWR_FLAG: +5V (источники - диоды D110/D30, пассивные) и GND (после смены типа GND у USB_B_Mini на passive)."
- note removed: "RESET шилда: D201 BAT54WS, анод - NRST, катод - вывод RESET разъёма. Кнопка шилда тянет RESET к GND -> NRST = Vf ~0.25-0.3 В при токе внутр. подтяжки (~40-80 мкА) < VIL(NRST) (DS13560 табл. 60). 5 В с шилда на RESET запирают диод и в NRST не попадают. Ограничение: шилд не видит сброс платы (вывод RESET разъёма не повторяет уровень NRST)."
- note removed: "VIN: D200 B120 от +5V, катод к VIN шилда. Шилд с собственным питанием на VIN (CNC Shield, GSM) не может подать напряжение в +5V платы и в USB-хост (обратный ток блокируется диодом). На VIN платы = +5V - Vf (~0.3-0.5 В). Внешнее питание платы через VIN не предусмотрено."
- note removed: "Гребёнки логического анализатора, 1x27 каждая (одинаковые, по левому и правому краю платы, подпись каждого вывода - на шелкографии): J205 J_LA_R (цифровой ряд Uno): SCL, SDA, AREF, GND, D13..D8, D7..D0 (порядок IOH+IOL), GND, SPI2 SCK/MISO/MOSI, W_CS, W_INT, U1_TX, U1_RX, GND. J204 J_LA_L (POWER/ANALOG): GND, 3V3, NRST, 5V, GND, VIN, A0..A5, GND, FL_CS, SD_CS, CARD_DET, W_RST, LED0, LED1, BTN, PO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"

Commit message: feat(schematic): add MPN/LCSC fields and fix Q201 pinout
Подготовка к заказу сборки на JLCPCB:
- всем монтируемым символам добавлено скрытое поле LCSC (коды
  проверены через API JLCPCB, по возможности Basic);
- LSE Y101: Epson FC-135 CL 7 пФ (Q13FC13500002), C106/C108 6.8p C0G,
  footprint под ручную пайку; в SDK нужен LSEDRV=10;
- бусины: FB101/FB401 GZ2012D601TF, FB301 BLM21PG221SN1D (2 А);
- Y401 25 МГц X49SD25MSD2SC (CL 20 пФ), C401/C402 27p -> 33p;
- Y201 8 МГц X49SD8MSD2SC, нагрузочные 22p оставлены (предел F103
  25 пФ, сдвиг частоты для USB FS несущественен);
- C505 100n на ~CARD_DET (антидребезг), ссылка на чертёж Hirose.

Исправления:
- Q201: символ SS9013 с распиновкой TO-92 (1=E 2=B 3=C) стоял на
  footprint SOT-23 (1=B 2=E 3=C) - транзистор встал бы неправильно.
  Заменён на MMBT3904 (SOT-23, Basic), цепи B/E/C сохранены;
- лист leds переведён с 1206 на 0805, R701/R702 630 -> 680 Ом
  (630 нет в E24), LD702 ORANGE -> RED;
- C301 (DNP) получил номинал 4.7n, опечатка 25Mhz в Y401.

ERC: 0 ошибок, 0 предупреждений.
Parts:
- D801: LCSC (none) -> C134421
- D802: LCSC (none) -> C124205
- J801: LCSC (none) -> C2905418
- J802, J803: LCSC (none) -> C42431840
- J804: LCSC (none) -> C40877
- JP801: LCSC (none) -> C225519
- R801, R802, R803: LCSC (none) -> C17477
Changed lines of the file:
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@@
+			)
+		)
+		(property "LCSC" "C42431840"
+			(at 101.6 106.68 0)
+			(hide yes)
+			(show_name no)
+			(do_not_autoplace no)
+			(effects
+				(font
+					(size 1.27 1.27)
+				)
 			)
 		)
@@
 			)
 		)
+		(property "LCSC" "C42431840"
+			(at 101.6 76.2 0)
+			(hide yes)
+			(show_name no)
+			(do_not_autoplace no)
+			(effects
+				(font
+					(size 1.27 1.27)
+				)
+			)
+		)
 		(pin "1"
 		)
@@
 			)
 		)
+		(property "LCSC" "C2905418"
+			(at 101.6 40.64 0)
+			(hide yes)
+			(show_name no)
+			(do_not_autoplace no)
+			(effects
+				(font
+					(size 1.27 1.27)
+				)
+			)
+		)
 		(pin "1"
 		)
@@
 			)
 		)
+		(property "LCSC" "C225519"
+			(at 213.36 177.8 0)
+			(hide yes)
+			(show_name no)
+			(do_not_autoplace no)
+			(effects
+				(font
+					(size 1.27 1.27)
+				)
+			)
+		)
 		(pin "1"
 		)
@@
 			)
 		)
+		(property "LCSC" ""
+			(at 254 73.66 0)
+			(hide yes)
+			(show_name no)
+			(do_not_autoplace no)
+			(effects
+				(font
+					(size 1.27 1.27)
+				)
+			)
+		)
 		(pin "1"
 		)
@@
 			)
 		)
+		(property "LCSC" ""
+			(at 182.88 73.66 0)
+			(hide yes)
+			(show_name no)
+			(do_not_autoplace no)
+			(effects
+				(font
+					(size 1.27 1.27)
+				)
+			)
+		)
 		(pin "1"
 		)
@@
 			)
 		)
+		(property "LCSC" "C40877"
+			(at 101.6 134.62 0)
+			(hide yes)
+			(show_name no)
+			(do_not_autoplace no)
+			(effects
+				(font
+					(size 1.27 1.27)
+				)
+			)
+		)
 		(pin "1"
 		)
@@
 			)
 		)
+		(property "LCSC" "C124205"
+			(at 157.48 177.8 0)
+			(hide yes)
+			(show_name no)
+			(do_not_autoplace no)
+			(effects
+				(font
+					(size 1.27 1.27)
+				)
+			)
+		)
 		(pin "1"
 		)
@@
 			)
 		)
+		(property "LCSC" "C17477"
+			(at 157.48 200.66 0)
+			(hide yes)
+			(show_name no)
+			(do_not_autoplace no)
+			(effects
+				(font
+					(size 1.27 1.27)
+				)
+			)
+		)
 		(pin "1"
 		)
@@
 			)
 		)
+		(property "LCSC" "C134421"
+			(at 157.48 165.1 0)
+			(hide yes)
+			(show_name no)
+			(do_not_autoplace no)
+			(effects
+				(font
+					(size 1.27 1.27)
+				)
+			)
+		)
 		(pin "1"
 		)
@@
 			)
 		)
+		(property "LCSC" "C17477"
+			(at 157.48 190.5 0)
+			(hide yes)
+			(show_name no)
+			(do_not_autoplace no)
+			(effects
+				(font
+					(size 1.27 1.27)
+				)
+			)
+		)
 		(pin "1"
 		)
@@
 			(at 157.48 210.82 0)
 			(hide yes)
+			(show_name no)
+			(do_not_autoplace no)
+			(effects
+				(font
+					(size 1.27 1.27)
+				)
+			)
+		)
+		(property "LCSC" "C17477"
+			(at 157.48 210.82 0)
+			(hide yes)

Commit message: refactor(pcb): reset routing, add power pins to J806, use GND on both inner layers
Плата откатена до расстановки: удалены все дорожки, переходные и полигоны.
Оба внутренних слоя (In1, In2) - сплошная общая GND.
Зафиксированы только контур платы, разъёмы Uno J801-J804, гребёнки
J805/J806 и крепёжные отверстия; остальные компоненты разблокированы
и оставлены на своих местах для ручной трассировки.

Схема: на гребёнке J806 вывод 3 (был AREF) -> +3.3V, вывод 27 (был GND)
-> +5V. Теперь на обеих гребёнках есть GND, +3.3V и +5V. AREF остаётся
только на разъёме Uno J801. ERC 0, DRC с паритетом схемы - 0 расхождений.
Connections:
- net +3.3V: now also J806.3 (Pin_3)
- net +5V: now also J806.27 (Pin_27)
- net AREF: no longer J806.3 (Pin_3)
- net GND: no longer J806.27 (Pin_27)
Other:
- note added: "Гребёнки логического анализатора, 1x27 каждая (одинаковые, по левому и правому краю платы, подпись каждого вывода - на шелкографии): J806 J_LA_R (цифровой ряд Uno): SCL, SDA, 3V3, GND, D13..D8, D7..D0 (порядок IOH+IOL), GND, SPI2 SCK/MISO/MOSI, W_CS, W_INT, U1_TX, U1_RX, 5V. На обеих гребёнках есть GND, 3V3 и 5V; AREF на гребёнку не выведен (только на J801). J805 J_LA_L (POWER/ANALOG): GND, 3V3, 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"
- note removed: "Гребёнки логического анализатора, 1x27 каждая (одинаковые, по левому и правому краю платы, подпись каждого вывода - на шелкографии): J806 J_LA_R (цифровой ряд Uno): SCL, SDA, AREF, GND, D13..D8, D7..D0 (порядок IOH+IOL), GND, SPI2 SCK/MISO/MOSI, W_CS, W_INT, U1_TX, U1_RX, GND. J805 J_LA_L (POWER/ANALOG): GND, 3V3, NRST, 5V, GND, VIN, A0..A5, GND, FL_CS, SD_CS, CARD_DET, W_RST, LED0, LED1, BTN, PO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"
Changed lines of the file:
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@@
 		(date "2026-10-18")
 	)
-	(text "Гребёнки логического анализатора, 1x27 каждая (одинаковые, по левому и правому краю платы,\nподпись каждого вывода - на шелкографии):\nJ806 J_LA_R (цифровой ряд Uno): SCL, SDA, AREF, GND, D13..D8, D7..D0 (порядок IOH+IOL),\n  GND, SPI2 SCK/MISO/MOSI, W_CS, W_INT, U1_TX, U1_RX, GND.\nJ805 J_LA_L (POWER/ANALOG): GND, 3V3, NRST, 5V, GND, VIN, A0..A5, GND, FL_CS, SD_CS, CARD_DET,\n  W_RST, LED0, LED1, BTN, POT, PF0, PF1, SWCLK(МК), SWDIO(МК), GND, GND.\nШина SPI2 общая для W5500, W25Q32 и microSD: SCK/MISO/MOSI выведены один раз (на J_LA_R),\nCS флэш/SD и детект - на J_LA_L. Свободных GPIO у МК в LQFP-48 только два (PF0, PF1);\nоставшиеся места - GND и SWD со стороны МК.\nU1_TX = PA9 (МК -> RXD FT232), U1_RX = PA10 (TXD FT232 -> МК)."
+	(text "Гребёнки логического анализатора, 1x27 каждая (одинаковые, по левому и правому краю платы,\nподпись каждого вывода - на шелкографии):\nJ806 J_LA_R (цифровой ряд Uno): SCL, SDA, 3V3, GND, D13..D8, D7..D0 (порядок IOH+IOL),\n  GND, SPI2 SCK/MISO/MOSI, W_CS, W_INT, U1_TX, U1_RX, 5V.\nНа обеих гребёнках есть GND, 3V3 и 5V; AREF на гребёнку не выведен (только на J801).\nJ805 J_LA_L (POWER/ANALOG): GND, 3V3, NRST, 5V, GND, VIN, A0..A5, GND, FL_CS, SD_CS, CARD_DET,\n  W_RST, LED0, LED1, BTN, POT, PF0, PF1, SWCLK(МК), SWDIO(МК), GND, GND.\nШина SPI2 общая для W5500, W25Q32 и microSD: SCK/MISO/MOSI выведены один раз (на J_LA_R),\nCS флэш/SD и детект - на J_LA_L. Свободных GPIO у МК в LQFP-48 только два (PF0, PF1);\nоставшиеся места - GND и SWD со стороны МК.\nU1_TX = PA9 (МК -> RXD FT232), U1_RX = PA10 (TXD FT232 -> МК)."
 		(exclude_from_sim no)
 		(at 279.4 119.38 0)
@@
 		)
 	)
-	(label "AREF"
-		(at 238.76 45.72 180)
-		(effects
-			(font
-				(size 1.27 1.27)
+	(symbol
+		(lib_id "power:+3.3V")
+		(at 238.76 45.72 90)
+		(unit 1)
+		(body_style 1)
+		(exclude_from_sim no)
+		(in_bom yes)
+		(on_board yes)
+		(in_pos_files yes)
+		(dnp no)
+		(property "Reference" "#PWR0152"
+			(at 171.45 43.18 90)
+			(hide yes)
+			(show_name no)
+			(do_not_autoplace no)
+			(effects
+				(font
+					(size 1.27 1.27)
+				)
+			)
+		)
+		(property "Value" "+3.3V"
+			(at 162.56 43.18 90)
+			(show_name no)
+			(do_not_autoplace no)
+			(effects
+				(font
+					(size 1.27 1.27)
+				)
+				(justify left)
+			)
+		)
+		(property "Footprint" ""
+			(at 238.76 45.72 0)
+			(hide yes)
+			(show_name no)
+			(do_not_autoplace no)
+			(effects
+				(font
+					(size 1.27 1.27)
+				)
+			)
+		)
+		(property "Datasheet" ""
+			(at 238.76 45.72 0)
+			(hide yes)
+			(show_name no)
+			(do_not_autoplace no)
+			(effects
+				(font
+					(size 1.27 1.27)
+				)
+			)
+		)
+		(property "Description" "Power symbol creates a global label with name \"+3.3V\""
+			(at 238.76 45.72 0)
+			(hide yes)
+			(show_name no)
+			(do_not_autoplace no)
+			(effects
+				(font
+					(size 1.27 1.27)
+				)
+			)
+		)
+		(pin "1"
+		)
+		(instances
+			(project "g0_dev_board"
+				(path "/997acf0a-b54e-4c77-ad84-80f8d6e2dc27/5c8f8cfd-1030-4022-9071-e1993a429931"
+					(reference "#PWR0152")
+					(unit 1)
+				)
 			)
-			(justify right bottom)
 		)
 	)
@@
 	)
 	(symbol
-		(lib_id "power:GND")
-		(at 238.76 106.68 270)
+		(lib_id "power:+5V")
+		(at 238.76 106.68 90)
 		(unit 1)
 		(body_style 1)
@@
 		(in_pos_files yes)
 		(dnp no)
-		(property "Reference" "#PWR0149"
-			(at 232.41 106.68 90)
+		(property "Reference" "#PWR0151"
+			(at 171.45 48.26 90)
 			(hide yes)
 			(show_name no)
@@
 			)
 		)
-		(property "Value" "GND"
-			(at 233.68 106.68 90)
-			(hide yes)
+		(property "Value" "+5V"
+			(at 162.56 48.26 90)
 			(show_name no)
 			(do_not_autoplace no)
@@
 			)
 		)
-		(property "Description" "Power symbol creates a global label with name \"GND\" , ground"
+		(property "Description" "Power symbol creates a global label with name \"+5V\""
 			(at 238.76 106.68 0)
 			(hide yes)
@@
 			(project "g0_dev_board"
 				(path "/997acf0a-b54e-4c77-ad84-80f8d6e2dc27/5c8f8cfd-1030-4022-9071-e1993a429931"
-					(reference "#PWR0149")
+					(reference "#PWR0151")
 					(unit 1)
 				)
